File: kicad/front/SUPER_UART_front.kicad_pcb (KiCad board)
At the start: 2 copper layers, 100 x 35 mm, 141 parts, among them CON1 UART A, CON2 UART B, CON3 UART C, CON4 UART D, CON5 RS232, CON6 UART A, Q1 PDTA143ZT, SW1 5V, SW10 TX, SW11 ISO, SW12 I2C, SW13 SPI, SW14 I2C, SW15 SPI, SW16 DTR, SW17 RTS, SW18 SPY, SW19 BOOT, SW2 3V3, SW3 2V5, SW4 1V8, SW5 5V, SW6 3V3, SW7 2V5, SW8 1V8, SW9 RX, U1 SN74LVC2T45DCTT, U10 MAX3243EIPW, U11 STM32F030C6T6, U2 SN74LVC2T45DCTT, U3 SN74LVC2T45DCTT, U4 SN74LVC2T45DCTT, U5 SN74LVC2T45DCTT, U6 SN74LVC2T45DCTT, U7 SN74LVC2T45DCTT, U8 SN74LVC2T45DCTT, U9 74HC595D

Commit message: Working on schematic
Parts:
- removed D52, D53: BAS70, SOT23-3_N
- removed U2: SN74LVC2T45DCTT, niceSemiconductors:TI_SSOP-8_N
- added C26: 100n, 0603_N, B.Cu at (153.3, 127.0)
- added C27: 100n, 0603_N, B.Cu at (145.5, 134.4)
- added C28: 100n, 0603_N, B.Cu at (154.0, 123.3)
- added C29: 100n, 0603_N, B.Cu at (149.9, 127.0)
- added C30: 100n, 0603_N, B.Cu at (142.1, 134.9)
- added C31: 100n, 0603_N, B.Cu at (146.4, 130.7)
- added C32: 100n, 0603_N, B.Cu at (150.5, 123.3)
- added C33: 100n, 0603_N, B.Cu at (154.0, 119.6)
- added C34: 100n, 0603_N, B.Cu at (138.6, 134.9)
- added C35: 100n, 0603_N, B.Cu at (186.6, 123.3)
- added C36: 100n, 0603_N, B.Cu at (181.1, 123.8)
- added C37: 27p, 0603_N, B.Cu at (174.8, 147.8)
- added C51: 27p, 0603_N, B.Cu at (181.0, 139.5)
- added Q2: PDTA143ZT, niceSemiconductors:SOT23-3_N, B.Cu at (174.7, 121.3)
- added Q3: PDTA143ZT, niceSemiconductors:SOT23-3_N, B.Cu at (164.7, 129.5)
- added Q4: 12MHz, XT3.2x2.5_N, B.Cu at (152.8, 136.8)
- added R11: R, 0603_R_N, B.Cu at (176.2, 132.1)
- added R12: R, 0603_R_N, B.Cu at (186.6, 119.6)
- added R13: 0R, 0603_R_N, B.Cu at (178.3, 143.8)
- added R14: R, 0603_R_N, B.Cu at (146.4, 127.0)
- added R15: R, 0603_R_N, B.Cu at (143.0, 127.5)
- added R16: R, 0603_R_N, B.Cu at (139.5, 123.8)
- added R17: R, 0603_R_N, B.Cu at (138.6, 131.2)
- added RN9: R, pnRLC:4x0603_N, B.Cu at (135.6, 124.4)
- added T1: DMG1012UW-7, niceSemiconductors:SC70-3_N, B.Cu at (181.9, 119.7)
- added T2: DMG1012UW-7, niceSemiconductors:SC70-3_N, B.Cu at (142.4, 119.7)
- added T3: DMG1012UW-7, niceSemiconductors:SC70-3_N, B.Cu at (136.4, 119.7)
- added U13: 74HC08P, niceSemiconductors:TSSOP-14_N, B.Cu at (154.3, 89.0)
- added U14: 74HC08P, niceSemiconductors:TSSOP-14_N, B.Cu at (131.6, 98.9)
- added U17: 74LVC1G125SE-7, niceSemiconductors:SC70-5_N, B.Cu at (172.4, 128.0)
- added U18: 74LVC1G02GW, niceSemiconductors:SC70-5_N, B.Cu at (171.7, 132.2)
- added U20: 74LVC8T245PW, TI_TSSOP-24_N, B.Cu at (165.9, 121.9)
- added U21: 74LVC8T245PW, TI_TSSOP-24_N, B.Cu at (128.9, 130.2)
- added U22: 74LVC8T245PW, TI_TSSOP-24_N, B.Cu at (128.9, 121.9)
- C5: moved to F.Cu
- MECH1: value dummy -> case; footprint niceMechanical:dummy -> dummy
- MH1, MH2: footprint niceMechanical:mounting_hole_3.2_7.5_plated -> mounting_hole_3.2_7.5_plated
- R3, R4: value R -> 10k
- U1: value SN74LVC2T45DCTT -> 74LVC1T45GW; footprint niceSemiconductors:TI_SSOP-8_N -> SC70-6_N
- U3, U4, U5, U6, U7, U8: value SN74LVC2T45DCTT -> 74LVC2T45DCU; footprint niceSemiconductors:TI_SSOP-8_N -> niceSemiconductors:TI_VSSOP-8_N
- U9: footprint SOIC-16_N -> niceSemiconductors:TSSOP-16_N
- moved TP5 75.2 mm to (162.1, 150.1)
- moved C18 75.1 mm to (177.6, 126.7)
- moved TP4 70.2 mm to (168.1, 145.5)
- moved R6 66.6 mm to (135.2, 128.7)
- moved R5 65.9 mm to (181.1, 127.5)
- moved TP3 64.8 mm to (163.5, 145.5)
- moved TP2 60.9 mm to (169.7, 140.0)
- moved U9 60.1 mm to (96.1, 77.3), turned to 90 degrees
- moved Q1 59.7 mm to (166.0, 150.0)
- moved C20 58.8 mm to (171.4, 147.8)
- moved TP1 57.3 mm to (173.7, 140.0)
- moved R3 51.4 mm to (174.8, 144.1)
- moved C19 41.5 mm to (171.4, 144.1)
- moved D51 30.2 mm to (177.3, 140.0)
- moved R2 28.7 mm to (139.5, 127.5)
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Connections:
- net CTS_B renamed /SUPER_UART_front_UART234/CTS_B_VDD
- net CTS_C renamed /SUPER_UART_front_UART234/CTS_C_VDD
- net CTS_D renamed /SUPER_UART_front_UART234/CTS_D_VDD
- net DCD_A_ISO renamed /SUPER_UART_front_UART1/DCD_D_VDDA
- net DSR_A_ISO renamed /SUPER_UART_front_UART1/DSR_D_VDDA
- net DTR_B renamed /SUPER_UART_front_UART234/DTR_B_VDD
- net DTR_C renamed /SUPER_UART_front_UART234/DTR_C_VDD
- net DTR_D renamed /SUPER_UART_front_UART234/DTR_D_VDD
- net FTDI_PWREN renamed PWREN
- net FT_CTS_B renamed /SUPER_UART_front_UART234/CTS_B
- net FT_CTS_C renamed /SUPER_UART_front_UART234/CTS_C
- net FT_CTS_D renamed /SUPER_UART_front_UART234/CTS_D
- net FT_DTR_B renamed /SUPER_UART_front_UART234/DTR_B
- net FT_DTR_C renamed /SUPER_UART_front_UART234/DTR_C
- net FT_DTR_D renamed /SUPER_UART_front_UART234/DTR_D
- net RI_A_ISO renamed /SUPER_UART_front_UART1/RI_D_VDDA
- net RS_CTS_ISO renamed /SUPER_UART_front_UART1/CTS_232
- net RS_DCD_ISO renamed /SUPER_UART_front_UART1/DCD_232
- net RS_DSR_ISO renamed /SUPER_UART_front_UART1/DSR_232
- net RS_DTR_ISO renamed /SUPER_UART_front_UART1/DTR_232
- net RS_RI_ISO renamed /SUPER_UART_front_UART1/RI_232
- net RS_RTS_ISO renamed /SUPER_UART_front_UART1/RTS_232
- net RS_RXD_ISO renamed /SUPER_UART_front_UART1/RXD_232
- net RS_TXD_ISO renamed /SUPER_UART_front_UART1/TXD_232
- net RXD_B renamed /SUPER_UART_front_UART234/RXD_B_VDD
- net RXD_C renamed /SUPER_UART_front_UART234/RXD_C_VDD
- net RXD_D renamed /SUPER_UART_front_UART234/RXD_D_VDD
- net TXD_B renamed /SUPER_UART_front_UART234/TXD_B_VDD
- net TXD_C renamed /SUPER_UART_front_UART234/TXD_C_VDD
- net TXD_D renamed /SUPER_UART_front_UART234/TXD_D_VDD
- C17 pad 1: ISO_VDD -> VDDA
- C17 pad 2: ISO_GND -> GND
- C22 pad 1: ISO_3V3 -> +3V3
- C22 pad 2: ISO_GND -> GND
- C24 pad 2: ISO_GND -> GND
- C25 pad 2: ISO_GND -> GND
- C4 pad 1: ISO_VDD -> VDDA
- C4 pad 2: ISO_GND -> GND
- C5 pad 1: ISO_VDD -> VDDA
- C5 pad 2: ISO_GND -> GND
- C6 pad 1: ISO_3V3 -> +3V3
- C6 pad 2: ISO_GND -> GND
- C7 pad 1: ISO_3V3 -> VDDA
- C7 pad 2: ISO_GND -> GND
- CON1 pad 1: DTR_A_ISO -> /SUPER_UART_front_UART1/DTR_D_VDDA
- CON1 pad 2: RXD_A_ISO -> /SUPER_UART_front_UART1/RXD_D_VDDA
- CON1 pad 3: TXD_A_ISO -> /SUPER_UART_front_UART1/TXD_D_VDDA
- CON1 pad 4: ISO_VDD -> VDDA
- CON1 pad 5: CTS_A_ISO -> /SUPER_UART_front_UART1/CTS_D_VDDA
- CON1 pad 6: ISO_GND -> GND
- CON5 pad 5: ISO_GND -> GND
- CON6 pad 10: ISO_GND -> GND
- CON6 pad 3: RTS_A_ISO -> /SUPER_UART_front_UART1/RTS_D_VDDA
- CON6 pad 4: RXD_A_ISO -> /SUPER_UART_front_UART1/RXD_D_VDDA
- CON6 pad 5: CTS_A_ISO -> /SUPER_UART_front_UART1/CTS_D_VDDA
- CON6 pad 6: TXD_A_ISO -> /SUPER_UART_front_UART1/TXD_D_VDDA
- CON6 pad 8: DTR_A_ISO -> /SUPER_UART_front_UART1/DTR_D_VDDA
- CON6 pad 9: ISO_VDD -> VDDA
- D1 pad 1: DTR_A_ISO -> /SUPER_UART_front_UART1/DTR_D_VDDA
- D1 pad 2: TXD_A_ISO -> /SUPER_UART_front_UART1/TXD_D_VDDA
- D1 pad 3: ISO_GND -> GND
- D12 pad 2: ISO_3V3 -> +3V3
- D2 pad 1: RXD_A_ISO -> /SUPER_UART_front_UART1/RXD_D_VDDA
- D2 pad 2: CTS_A_ISO -> /SUPER_UART_front_UART1/CTS_D_VDDA
- D2 pad 3: ISO_GND -> GND
- D25 pad 2: RTS_A_ISO -> /SUPER_UART_front_UART1/RTS_D_VDDA
- D25 pad 3: ISO_GND -> GND
- D26 pad 1: CTS_A_ISO -> /SUPER_UART_front_UART1/CTS_D_VDDA
- D26 pad 3: ISO_GND -> GND
- D27 pad 1: DTR_A_ISO -> /SUPER_UART_front_UART1/DTR_D_VDDA
- D27 pad 2: TXD_A_ISO -> /SUPER_UART_front_UART1/TXD_D_VDDA
- D27 pad 3: ISO_GND -> GND
- D28 pad 1: RXD_A_ISO -> /SUPER_UART_front_UART1/RXD_D_VDDA
- D28 pad 3: ISO_GND -> GND
- D29 pad 2: ISO_3V3 -> +3V3
- D30 pad 2: ISO_3V3 -> +3V3
- D31 pad 2: ISO_3V3 -> +3V3
- D32 pad 2: ISO_3V3 -> +3V3
- D51 pad 1: FTDI_DTR_A_ISO1 -> RST
- D51 pad 3: Net-(D48-Pad1) -> Net-(D51-Pad3)
- D9 pad 2: ISO_3V3 -> +3V3
- MH1 pad 1: ISO_GND -> GND
- MH2 pad 1: ISO_GND -> GND
- Q1 pad 1: Net-(D53-Pad3) -> Net-(D51-Pad3)
- R1 pad 2: ISO_3V3 -> +3V3
- R10 pad 1: TXD_A_LED -> (no net)
- R2 pad 2: ISO_3V3 -> +3V3
- R3 pad 1: FTDI_DTR_A_ISO1 -> ISO_GND
- R3 pad 2: (no net) -> BOOT0
- R4 pad 1: FTDI_RTS_A_ISO1 -> Net-(D48-Pad1)
- R4 pad 2: (no net) -> +3V3
- R6 pad 1: ISO_GND -> Net-(D49-Pad1)
- R6 pad 2: BOOT0 -> +3V3
- R7 pad 1: (no net) -> /SUPER_UART_front_UART1/DCD_D
- R8 pad 1: (no net) -> /SUPER_UART_front_UART1/DTR_D
- R9 pad 1: RXD_A_LED -> (no net)
- RN1 pad 1: DTR_A_ISO -> /SUPER_UART_front_UART1/TXD_D_VDDA
- RN1 pad 2: TXD_A_ISO -> /SUPER_UART_front_UART1/DTR_D_VDDA
- RN1 pad 3: RXD_A_ISO -> /SUPER_UART_front_UART1/RTS_D_VDDA
- RN1 pad 4: CTS_A_ISO -> (no net)
- RN8 pad 1: (no net) -> /SUPER_UART_front_UART1/RI_D
- RN8 pad 2: (no net) -> /SUPER_UART_front_UART1/CTS_D
- RN8 pad 3: (no net) -> /SUPER_UART_front_UART1/RTS_D
- RN8 pad 4: (no net) -> /SUPER_UART_front_UART1/DSR_D
- SW16 pad 2: ISO_GND -> GND
- SW17 pad 2: ISO_GND -> GND
- SW19 pad 1: Net-(D53-Pad3) -> Net-(D51-Pad3)
- U1 pad 1: ISO_VDD -> +3V3
- U1 pad 2: Net-(RN1-Pad7) -> GND
- U1 pad 3: Net-(RN1-Pad8) -> (no net)
- U1 pad 4: ISO_GND -> Net-(R17-Pad1)
- U1 pad 5: ISO_GND -> (no net)
- U1 pad 6: FT_DTR_A_ISO -> VDDA
- U10 pad 12: FT_DTR_A_ISO -> /SUPER_UART_front_UART1/DTR_D1
- U10 pad 13: FT_TXD_A_ISO -> (no net)
- U10 pad 14: (no net) -> /SUPER_UART_front_UART1/RTS_D1
- U10 pad 15: (no net) -> /SUPER_UART_front_UART1/RI_D2
- U10 pad 16: (no net) -> /SUPER_UART_front_UART1/CTS_D2
- U10 pad 17: (no net) -> /SUPER_UART_front_UART1/RXD_D2
- U10 pad 18: (no net) -> /SUPER_UART_front_UART1/DCD_D2
- U10 pad 19: (no net) -> /SUPER_UART_front_UART1/DSR_D2
- U10 pad 22: ISO_3V3 -> +3V3
- U10 pad 23: ISO_3V3 -> +3V3
- U10 pad 25: ISO_GND -> GND
- U10 pad 26: ISO_3V3 -> +3V3
- U11 pad 29: (no net) -> Net-(R13-Pad2)
- U11 pad 5: (no net) -> Net-(C51-Pad1)
- U11 pad 6: (no net) -> Net-(C37-Pad1)
- U9 pad 1: RXD_A_LED -> (no net)
- U9 pad 15: TXD_A_LED -> (no net)
Routing:
- net /SUPER_UART_front_UART1/CTS_D_VDDA: track 0.00 -> 31.3 mm
- net /SUPER_UART_front_UART1/RXD_D_VDDA: track 0.00 -> 27.7 mm, vias 0 -> 1
- net /SUPER_UART_front_UART1/TXD_D_VDDA: track 0.00 -> 24.7 mm
- net /SUPER_UART_front_UART1/DTR_D_VDDA: track 0.00 -> 24.6 mm
- net GND: track 39.5 -> 61.4 mm, vias 12 -> 16
- net ISO_GND: track 15.6 -> 0.00 mm, vias 4 -> 0
- net +3V3: track 16.3 -> 30.7 mm, vias 6 -> 7
- net VDDA: track 0.00 -> 13.8 mm, vias 0 -> 2
- net RXD_A_ISO: track 10.4 -> 0.00 mm
- net ISO_VDD: track 9.22 -> 0.00 mm, vias 1 -> 0
- net CTS_A_ISO: track 7.80 -> 0.00 mm
- net DTR_A_ISO: track 5.86 -> 0.00 mm
- net TXD_A_ISO: track 5.52 -> 0.00 mm
- net ISO_3V3: track 5.43 -> 0.00 mm, vias 2 -> 0
- net Net-(RN1-Pad8): track 4.81 -> 0.60 mm
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
Commit message: Working on schematic
Parts:
- removed C51: 27p, 0603_N
- removed D14, D18, D22: RXD, pnSemiconductor:LED0603_R
- removed D15, D19, D23: TXD, pnSemiconductor:LED0603_R
- removed D16, D20, D24: CTS, pnSemiconductor:LED0603_R
- removed D17, D21: DTR, pnSemiconductor:LED0603_R
- removed D25, D26, D27, D28: PESD5V2S2UT, SOT23-3_N
- removed D29: DSR, pnSemiconductor:LED0603_R
- removed D30: RTS, pnSemiconductor:LED0603_R
- removed D31: RI, pnSemiconductor:LED0603_R
- removed D32: DCD, pnSemiconductor:LED0603_R
- removed D33, D37: 5V, pnSemiconductor:LED_3.2x2
- removed D34, D38: 3V3, pnSemiconductor:LED_3.2x2
- removed D35, D39: 2V5, pnSemiconductor:LED_3.2x2
- removed D36, D40: 1V8, pnSemiconductor:LED_3.2x2
- removed D41: RX, pnSemiconductor:LED_3.2x2
- removed D42: TX, pnSemiconductor:LED_3.2x2
- removed D43: ISO, pnSemiconductor:LED_3.2x2
- removed D44, D46: I2C, pnSemiconductor:LED_3.2x2
- removed D45, D47: SPI, pnSemiconductor:LED_3.2x2
- removed D48: DTR, pnSemiconductor:LED_3.2x2
- removed D49: RTS, pnSemiconductor:LED_3.2x2
- removed D50: SPY, pnSemiconductor:LED_3.2x2
- removed D51: BAS70, SOT23-3_N
- removed T1, T2, T3: DMG1012UW-7, niceSemiconductors:SC70-3_N
- removed TP3: SWDCLK, pnConnector:TP_1mm
- removed TP4: RST, pnConnector:TP_1mm
- removed TP5: GND, pnConnector:TP_1mm
- removed U17: 74LVC1G125SE-7, niceSemiconductors:SC70-5_N
- removed U18: 74LVC1G02GW, niceSemiconductors:SC70-5_N
- removed U20, U21, U22: 74LVC8T245PW, TI_TSSOP-24_N
- added C38: 100n, 0603_N, B.Cu at (131.1, 157.0)
- added C39: 100n, 0603_N, B.Cu at (138.3, 155.2)
- added C40: 100n, 0603_N, B.Cu at (141.1, 147.4)
- added C41: 100n, 0603_N, B.Cu at (123.5, 166.3)
- added C42: 100n, 0603_N, B.Cu at (147.2, 143.1)
- added C43: 10n, 0603_N, B.Cu at (138.3, 151.5)
- added C44: 10u, niceRLC:0805_N, B.Cu at (134.5, 152.3)
- added C45: 100n, 0603_N, B.Cu at (129.4, 161.1)
- added C46: 100n, 0603_N, B.Cu at (144.5, 146.8)
- added C47: 1u, niceRLC:0603_N, B.Cu at (150.7, 141.9)
- added C48: 100n, 0603_N, F.Cu at (125.9, 162.0)
- added CON7: UART B, pnConnector:NIGINI_NCDW-06, B.Cu at (109.6, 145.5)
- added CON8: UART C, pnConnector:NIGINI_NCDW-06, F.Cu at (118.6, 145.5)
- added LED1: 5V_1, pnSemiconductor:LED_3.2x2, B.Cu at (176.1, 106.2)
- added LED10: 3V3_2, pnSemiconductor:LED_3.2x2, B.Cu at (189.5, 84.8)
- added LED11: 2V5_2, pnSemiconductor:LED_3.2x2, B.Cu at (197.8, 79.7)
- added LED12: 1V8_2, pnSemiconductor:LED_3.2x2, B.Cu at (171.8, 105.6)
- added LED13: I2C_A, pnSemiconductor:LED_3.2x2, B.Cu at (174.0, 102.0)
- added LED14: SPI_A, pnSemiconductor:LED_3.2x2, B.Cu at (189.5, 88.3)
- added LED15: I2C_B, pnSemiconductor:LED_3.2x2, B.Cu at (185.2, 92.5)
- added LED16: SPI_B, pnSemiconductor:LED_3.2x2, B.Cu at (178.4, 99.2)
- added LED17: EN_A, pnSemiconductor:LED_3.2x2, B.Cu at (167.4, 110.5)
- added LED18: EN_B, pnSemiconductor:LED_3.2x2, B.Cu at (193.9, 88.3)
- added LED19: EN_C, pnSemiconductor:LED_3.2x2, B.Cu at (193.9, 84.8)
- added LED2: 3V3_1, pnSemiconductor:LED_3.2x2, B.Cu at (187.6, 96.0)
- added LED20: EN_D, pnSemiconductor:LED_3.2x2, B.Cu at (198.2, 86.8)
- added LED21: DTR, pnSemiconductor:LED_3.2x2, B.Cu at (194.9, 137.0)
- added LED22: RTS, pnSemiconductor:LED_3.2x2, B.Cu at (207.0, 127.2)
- added LED23: RI, pnSemiconductor:LED0603_R, B.Cu at (168.0, 144.0)
- added LED24: CTS, pnSemiconductor:LED0603_R, B.Cu at (176.8, 143.7)
- added LED25: DSR, pnSemiconductor:LED0603_R, B.Cu at (171.6, 144.0)
- added LED26: DCD, pnSemiconductor:LED0603_R, B.Cu at (193.5, 143.6)
- added LED27: TXD, pnSemiconductor:LED0603_R, B.Cu at (74.3, 167.3)
- added LED28: RXD, pnSemiconductor:LED0603_R, B.Cu at (74.3, 170.1)
- added LED29: DTR, pnSemiconductor:LED0603_R, B.Cu at (69.9, 171.0)
- added LED3: 2V5_1, pnSemiconductor:LED_3.2x2, B.Cu at (171.8, 112.7)
- added LED30: RTS, pnSemiconductor:LED0603_R, B.Cu at (89.9, 153.6)
- added LED31: DTR, pnSemiconductor:LED0603_R, B.Cu at (78.3, 163.6)
- added LED32: CTS, pnSemiconductor:LED0603_R, B.Cu at (92.1, 149.3)
- added LED33: RXD, pnSemiconductor:LED0603_R, B.Cu at (83.0, 159.4)
- added LED34: TXD, pnSemiconductor:LED0603_R, B.Cu at (97.3, 145.6)
- added LED35: DTR, pnSemiconductor:LED0603_R, B.Cu at (152.1, 149.3)
- added LED36: CTS, pnSemiconductor:LED0603_R, B.Cu at (125.0, 152.9)
- added LED37: RXD, pnSemiconductor:LED0603_R, B.Cu at (158.3, 145.6)
- added LED38: TXD, pnSemiconductor:LED0603_R, B.Cu at (161.0, 141.9)
- added LED39: DTR, pnSemiconductor:LED0603_R, F.Cu at (148.6, 153.4)
- added LED4: 1V8_1, pnSemiconductor:LED_3.2x2, B.Cu at (182.7, 99.6)
- added LED40: CTS, pnSemiconductor:LED0603_R, F.Cu at (145.2, 157.1)
- added LED41: RXD, pnSemiconductor:LED0603_R, F.Cu at (133.8, 166.5)
- added LED42: TXD, pnSemiconductor:LED0603_R, F.Cu at (139.7, 165.1)
- added LED5: RX, pnSemiconductor:LED_3.2x2, B.Cu at (198.2, 83.2)
- added LED6: TX, pnSemiconductor:LED_3.2x2, B.Cu at (189.5, 91.8)
- added LED7: SPY, pnSemiconductor:LED_3.2x2, B.Cu at (183.3, 96.0)
- added LED8: ISO, pnSemiconductor:LED_3.2x2, B.Cu at (171.8, 109.2)
- added LED9: 5V_2, pnSemiconductor:LED_3.2x2, B.Cu at (178.4, 102.7)
- added Q10: 2N7002PS, niceSemiconductors:SC70-6_N, B.Cu at (127.3, 157.4)
- added Q11: N-MOS_small, SOT23-3_N, B.Cu at (140.4, 138.6)
- added Q5: 2N7002PS, niceSemiconductors:SC70-6_N, B.Cu at (51.4, 171.3)
- added Q6: N-MOS_small, SOT23-3_N, B.Cu at (69.2, 152.3)
- added Q7: PDTA143ZT, niceSemiconductors:SOT23-3_N, B.Cu at (122.0, 162.4)
- added Q8: 2N7002PS, niceSemiconductors:SC70-6_N, B.Cu at (137.2, 147.8)
- added Q9: PDTA143ZT, niceSemiconductors:SOT23-3_N, B.Cu at (116.1, 166.6)
- added R18: 10k, 0603_R_N, B.Cu at (90.4, 145.6)
- added R19: 10k, 0603_R_N, B.Cu at (98.3, 138.2)
- added R20: 4k7, 0603_R_N, B.Cu at (94.8, 141.9)
- added R21: 10k, 0603_R_N, B.Cu at (88.7, 149.9)
- added R22: 10k, 0603_R_N, B.Cu at (59.3, 170.9)
- added R23: 1k8, 0603_R_N, B.Cu at (78.1, 152.2)
- added R24: 3k9, 0603_R_N, B.Cu at (81.5, 148.5)
- added R25: 6k8, 0603_R_N, B.Cu at (87.0, 142.5)
- added R26: 10k, 0603_R_N, B.Cu at (91.4, 138.2)
- added R27: 5k6, 0603_R_N, B.Cu at (72.4, 156.2)
- added R28: 47k, 0603_R_N, B.Cu at (78.1, 148.5)
- added R29: 10k, 0603_R_N, B.Cu at (139.7, 162.2)
- added R30: R, 0603_R_N, B.Cu at (154.9, 145.6)
- added R31: R, 0603_R_N, B.Cu at (157.6, 141.9)
- added R32: R, 0603_R_N, B.Cu at (145.2, 154.2)
- added R33: R, 0603_R_N, B.Cu at (148.6, 150.5)
- added R34: 10k, 0603_R_N, B.Cu at (136.3, 163.6)
- added R35: 10k, 0603_R_N, B.Cu at (156.2, 138.2)
- added R36: R, 0603_R_N, B.Cu at (151.4, 145.6)
- added R37: 10k, 0603_R_N, B.Cu at (159.7, 138.2)
- added R38: 10k, 0603_R_N, B.Cu at (136.3, 159.9)
- added R39: R, 0603_R_N, B.Cu at (145.2, 150.5)
- added R40: 4k7, 0603_R_N, B.Cu at (130.4, 164.8)
- added R41: 10k, 0603_R_N, B.Cu at (154.1, 141.9)
- added R42: 1k8, 0603_R_N, B.Cu at (141.7, 154.8)
- added R43: 3k9, 0603_R_N, B.Cu at (148.0, 146.8)
- added R44: 6k8, 0603_R_N, B.Cu at (126.9, 165.7)
- added R45: 10k, 0603_R_N, F.Cu at (141.7, 158.5)
- added R46: 5k6, 0603_R_N, F.Cu at (134.6, 156.2)
- added R47: 47k, 0603_R_N, F.Cu at (152.8, 138.2)
- added U12: 74LVC8T245PW, TI_TSSOP-24_N, B.Cu at (110.9, 158.8)
- added U15: 74LVC1T45GW, SC70-6_N, F.Cu at (118.2, 156.6)
- added U16: LP2951CD, SOIC-8_N, F.Cu at (134.7, 140.6)
- added U2: MIC5504-3.3YM5-TR, niceSemiconductors:SOT23-5_N, B.Cu at (191.5, 80.1)
- C1, C11, C28, C8: value 100n -> 10u; footprint 0603_N -> niceRLC:0805_N
- C10, C13, C14, C15, C16, C6, C9: value 100n -> 1u
- C19: value 1u -> 100n
- C20: value 10n -> 100n
- C23, C24, C25: value 470n -> 100n
- C27, C7: value 100n -> 10n
- C31: value 100n -> 1u; footprint 0603_N -> niceRLC:0603_N
- C37: value 27p -> 100n
- C5, MH1, MH2, RN8: moved to B.Cu
- CON1: value UART A -> PIN-2x20; footprint pnConnector:NIGINI_NCDW-06 -> PIN-2x20_N; moved to B.Cu
- CON2: value UART B -> PIN-2x3; footprint pnConnector:NIGINI_NCDW-06 -> pnPinheaders:PIN3x2SMD; moved to B.Cu
- CON3: value UART C -> RS232; footprint pnConnector:NIGINI_NCDW-06 -> pnConnector:DB9MV; moved to B.Cu
- CON4: value UART D -> UART A; footprint pnConnector:NIGINI_NCDW-06 -> pnIDC:IDC10; moved to B.Cu
- CON5: value RS232 -> UART A; footprint pnConnector:DB9MV -> pnConnector:NIGINI_NCDW-06; moved to B.Cu
- CON6: value UART A -> UART D; footprint pnIDC:IDC10 -> pnConnector:NIGINI_NCDW-06; moved to B.Cu
- D1: value PESD5V2S2UT -> BAS70
- D10: value RXD -> PESD5V2S2UT; footprint pnSemiconductor:LED0603_R -> SOT23-3_N; moved to B.Cu
- D11: value TXD -> PESD5V2S2UT; footprint pnSemiconductor:LED0603_R -> SOT23-3_N; moved to B.Cu
- D12: value CTS -> PESD5V2S2UT; footprint pnSemiconductor:LED0603_R -> SOT23-3_N; moved to B.Cu
- D13, D9: value DTR -> PESD5V2S2UT; footprint pnSemiconductor:LED0603_R -> SOT23-3_N; moved to B.Cu
- Q3: value PDTA143ZT -> 2N7002PS; footprint niceSemiconductors:SOT23-3_N -> niceSemiconductors:SC70-6_N
- Q4: value 12MHz -> PDTA143ZT; footprint XT3.2x2.5_N -> niceSemiconductors:SOT23-3_N
- R1: footprint 0603_R_N -> pnRLC:0805_JUMPER
- R13: value 0R -> R
- R15, R2: value R -> 10k
- R3, R5: value 10k -> R
- RN2: value R -> N.C.
- RN5, RN7: footprint 4x0603_N -> pnRLC:4x0603_N; moved to B.Cu
- RN6: footprint 4x0603_N -> pnRLC:4x0603_N
- SW1: value 5V -> 5V_1; moved to B.Cu
- SW10: value TX -> 3V3_2; moved to B.Cu
- SW11: value ISO -> 2V5_2; moved to B.Cu
- SW12: value I2C -> 1V8_2; moved to B.Cu
- SW13: value SPI -> I2C_A; moved to B.Cu
- SW14: value I2C -> SPI_A; moved to B.Cu
- SW15: value SPI -> I2C_B; moved to B.Cu
- SW16: value DTR -> SPI_B; moved to B.Cu
- SW17: value RTS -> BOOT; moved to B.Cu
- SW18: value SPY -> DTR; moved to B.Cu
- SW19: value BOOT -> RTS; moved to B.Cu
- SW2: value 3V3 -> 3V3_1; moved to B.Cu
- SW3: value 2V5 -> 2V5_1; moved to B.Cu
- SW4: value 1V8 -> 1V8_1; moved to B.Cu
- SW5: value 5V -> RX; moved to B.Cu
- SW6: value 3V3 -> TX; moved to B.Cu
- SW7: value 2V5 -> SPY; moved to B.Cu
- SW8: value 1V8 -> ISO; moved to B.Cu
- SW9: value RX -> 5V_2; moved to B.Cu
- TP1: value 3V3 -> Testpoint
- TP2: value SWDIO -> Testpoint
- U1: value 74LVC1T45GW -> STM32F030C6T6; footprint SC70-6_N -> ST_LQFP48_ST_default
- U10: value MAX3243EIPW -> LP2951CD; footprint TSSOP-28_N -> SOIC-8_N
- U11: value STM32F030C6T6 -> 74HC595D; footprint ST_LQFP48_ST_default -> niceSemiconductors:TSSOP-16_N
- U13: value 74HC08P -> 74LVC2T45DCU; footprint niceSemiconductors:TSSOP-14_N -> niceSemiconductors:TI_VSSOP-8_N
- U14: value 74HC08P -> 74LVC1T45GW; footprint niceSemiconductors:TSSOP-14_N -> SC70-6_N
- U3: value 74LVC2T45DCU -> AP7333-33SAG-7; footprint niceSemiconductors:TI_VSSOP-8_N -> SOT23-3_N
- U4, U6: value 74LVC2T45DCU -> 74HC08P; footprint niceSemiconductors:TI_VSSOP-8_N -> niceSemiconductors:TSSOP-14_N
- U5: value 74LVC2T45DCU -> MAX3243EIPW; footprint niceSemiconductors:TI_VSSOP-8_N -> TSSOP-28_N
- U7, U8: value 74LVC2T45DCU -> 74LVC8T245PW; footprint niceSemiconductors:TI_VSSOP-8_N -> TI_TSSOP-24_N
- U9: value 74HC595D -> 74LVC1T45GW; footprint niceSemiconductors:TSSOP-16_N -> SC70-6_N
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Connections:
- C1 pad 1: VDD -> +5V
- C12 pad 1: VDD -> Net-(C12-Pad1)
- C12 pad 2: GND -> Net-(C12-Pad2)
- C13 pad 1: VDD -> +3V3
- C14 pad 1: VDD -> Net-(C14-Pad1)
- C14 pad 2: GND -> Net-(C14-Pad2)
- C15 pad 1: +3V3 -> Net-(C15-Pad1)
- C16 pad 1: +3V3 -> Net-(C16-Pad1)
- C17 pad 1: VDDA -> +3V3
- C19 pad 1: BOOT0 -> VDD1
- C19 pad 2: ISO_GND -> GND
- C20 pad 1: RST -> +3V3
- C20 pad 2: ISO_GND -> GND
- C21 pad 1: Net-(C21-Pad1) -> VDD1
- C21 pad 2: Net-(C21-Pad2) -> GND
- C22 pad 1: +3V3 -> VDD1
- C23 pad 1: Net-(C23-Pad1) -> VDD1
- C23 pad 2: Net-(C23-Pad2) -> GND
- C24 pad 1: Net-(C24-Pad1) -> +3V3
- C25 pad 1: Net-(C25-Pad1) -> VDD1
- C26 pad 1: VDDA -> +5V
- C27 pad 1: VDDA -> VDD1
- C27 pad 2: GND -> Net-(C27-Pad2)
- C28 pad 1: +3V3 -> VDD1
- C30 pad 1: +3V3 -> VDD1
- C31 pad 1: +3V3 -> Net-(C31-Pad1)
- C32 pad 1: +3V3 -> Net-(C32-Pad1)
- C34 pad 1: VDDA -> VDD2
- C35 pad 1: VDD -> +3V3
- C36 pad 1: +3V3 -> VDD2
- C37 pad 1: Net-(C37-Pad1) -> +3V3
- C4 pad 1: VDDA -> +3V3
- C5 pad 1: VDDA -> +3V3
- C6 pad 1: +3V3 -> /SUPER_UART_front_uC/BOOT0
- C7 pad 1: VDDA -> /SUPER_UART_front_uC/RST
- C8 pad 1: VDD -> +5V
- C9 pad 1: VDD -> +5V
- CON1 pad 1: /SUPER_UART_front_UART1/DTR_D_VDDA -> /EEDATA 
- CON1 pad 2: /SUPER_UART_front_UART1/RXD_D_VDDA -> /RXD_D 
- CON1 pad 3: /SUPER_UART_front_UART1/TXD_D_VDDA -> /RXD_C 
- CON1 pad 4: VDDA -> /TXD_D 
- CON1 pad 5: /SUPER_UART_front_UART1/CTS_D_VDDA -> /EECLK 
- CON1 pad 6: GND -> /RTS_D 
- CON2 pad 1: /SUPER_UART_front_UART234/DTR_B_VDD -> +3V3
- CON2 pad 2: /SUPER_UART_front_UART234/RXD_B_VDD -> /SUPER_UART_front_uC/SWDIO
- CON2 pad 3: /SUPER_UART_front_UART234/TXD_B_VDD -> /SUPER_UART_front_uC/RST
- CON2 pad 4: VDD -> /SUPER_UART_front_uC/SWDCLK
- CON2 pad 5: /SUPER_UART_front_UART234/CTS_B_VDD -> GND
- CON2 pad 6: GND -> (no net)
- CON3 pad 1: /SUPER_UART_front_UART234/DTR_C_VDD -> /SUPER_UART_front_RS232/DCD_232
- CON3 pad 2: /SUPER_UART_front_UART234/RXD_C_VDD -> /SUPER_UART_front_RS232/RXD_232
- CON3 pad 3: /SUPER_UART_front_UART234/TXD_C_VDD -> /SUPER_UART_front_RS232/TXD_232
- CON3 pad 4: VDD -> /SUPER_UART_front_RS232/DTR_232
- CON3 pad 5: /SUPER_UART_front_UART234/CTS_C_VDD -> GND
- CON3 pad 6: GND -> /SUPER_UART_front_RS232/DSR_232
- CON4 pad 1: /SUPER_UART_front_UART234/DTR_D_VDD -> /SUPER_UART_front_UART1/DSR_D_VDD1
- CON4 pad 2: /SUPER_UART_front_UART234/RXD_D_VDD -> /SUPER_UART_front_UART1/DCD_D_VDD1
- CON4 pad 3: /SUPER_UART_front_UART234/TXD_D_VDD -> /SUPER_UART_front_UART1/RTS_D_VDD1
- CON4 pad 4: VDD -> /SUPER_UART_front_UART1/RXD_D_VDD1
- CON4 pad 5: /SUPER_UART_front_UART234/CTS_D_VDD -> /SUPER_UART_front_UART1/CTS_D_VDD1
- CON4 pad 6: GND -> /SUPER_UART_front_UART1/TXD_D_VDD1
- CON5 pad 1: /SUPER_UART_front_UART1/DCD_232 -> /SUPER_UART_front_UART1/DTR_D_VDD1
- CON5 pad 2: /SUPER_UART_front_UART1/RXD_232 -> /SUPER_UART_front_UART1/RXD_D_VDD1
- CON5 pad 3: /SUPER_UART_front_UART1/TXD_232 -> /SUPER_UART_front_UART1/TXD_D_VDD1
- CON5 pad 4: /SUPER_UART_front_UART1/DTR_232 -> VDD1
- CON5 pad 5: GND -> /SUPER_UART_front_UART1/CTS_D_VDD1
- CON5 pad 6: /SUPER_UART_front_UART1/DSR_232 -> GND
- CON6 pad 1: /SUPER_UART_front_UART1/DSR_D_VDDA -> /SUPER_UART_front_UART1/DTR_B_VDD1
- CON6 pad 2: /SUPER_UART_front_UART1/DCD_D_VDDA -> /SUPER_UART_front_UART1/RXD_B_VDD1
- CON6 pad 3: /SUPER_UART_front_UART1/RTS_D_VDDA -> /SUPER_UART_front_UART1/TXD_B_VDD1
- CON6 pad 4: /SUPER_UART_front_UART1/RXD_D_VDDA -> VDD1
- CON6 pad 5: /SUPER_UART_front_UART1/CTS_D_VDDA -> /SUPER_UART_front_UART1/CTS_B_VDD1
- CON6 pad 6: /SUPER_UART_front_UART1/TXD_D_VDDA -> GND
- D1 pad 1: /SUPER_UART_front_UART1/DTR_D_VDDA -> /SUPER_UART_front_uC/RST
- D1 pad 2: /SUPER_UART_front_UART1/TXD_D_VDDA -> (no net)
- D1 pad 3: GND -> Net-(D1-Pad3)
- D10 pad 1: GND -> /SUPER_UART_front_UART234/DTR_A_VDD2
- D10 pad 2: Net-(D10-Pad2) -> /SUPER_UART_front_UART234/TXD_A_VDD2
- D11 pad 1: GND -> /SUPER_UART_front_UART234/RXD_A_VDD2
- D11 pad 2: Net-(D11-Pad2) -> /SUPER_UART_front_UART234/CTS_A_VDD2
- D12 pad 1: Net-(D12-Pad1) -> /SUPER_UART_front_UART234/DTR_C_VDD2
- D12 pad 2: +3V3 -> /SUPER_UART_front_UART234/TXD_C_VDD2
- D13 pad 1: Net-(D13-Pad1) -> /SUPER_UART_front_UART234/RXD_C_VDD2
- D13 pad 2: +3V3 -> /SUPER_UART_front_UART234/CTS_C_VDD2
- D2 pad 1: /SUPER_UART_front_UART1/RXD_D_VDDA -> /SUPER_UART_front_UART1/DSR_D_VDD1
- D2 pad 2: /SUPER_UART_front_UART1/CTS_D_VDDA -> /SUPER_UART_front_UART1/RTS_D_VDD1
- D3 pad 1: /SUPER_UART_front_UART234/DTR_B_VDD -> /SUPER_UART_front_UART1/CTS_D_VDD1
- D3 pad 2: /SUPER_UART_front_UART234/TXD_B_VDD -> /SUPER_UART_front_UART1/RI_D_VDD1
- D4 pad 1: /SUPER_UART_front_UART234/RXD_B_VDD -> /SUPER_UART_front_UART1/DTR_D_VDD1
- D4 pad 2: /SUPER_UART_front_UART234/CTS_B_VDD -> /SUPER_UART_front_UART1/TXD_D_VDD1
- D5 pad 1: /SUPER_UART_front_UART234/DTR_C_VDD -> /SUPER_UART_front_UART1/RXD_D_VDD1
- D5 pad 2: /SUPER_UART_front_UART234/TXD_C_VDD -> /SUPER_UART_front_UART1/DCD_D_VDD1
- D6 pad 1: /SUPER_UART_front_UART234/RXD_C_VDD -> /SUPER_UART_front_UART1/DTR_D_VDD1
- D6 pad 2: /SUPER_UART_front_UART234/CTS_C_VDD -> /SUPER_UART_front_UART1/TXD_D_VDD1
- D7 pad 1: /SUPER_UART_front_UART234/DTR_D_VDD -> /SUPER_UART_front_UART1/RXD_D_VDD1
- D7 pad 2: /SUPER_UART_front_UART234/TXD_D_VDD -> /SUPER_UART_front_UART1/CTS_D_VDD1
- D8 pad 1: /SUPER_UART_front_UART234/RXD_D_VDD -> /SUPER_UART_front_UART1/DTR_B_VDD1
- D8 pad 2: /SUPER_UART_front_UART234/CTS_D_VDD -> /SUPER_UART_front_UART1/TXD_B_VDD1
- D9 pad 1: Net-(D9-Pad1) -> /SUPER_UART_front_UART1/RXD_B_VDD1
- D9 pad 2: +3V3 -> /SUPER_UART_front_UART1/CTS_B_VDD1
- Q1 pad 1: Net-(D51-Pad3) -> Net-(D1-Pad3)
- Q1 pad 2: ISO_3V3 -> +3V3
- Q1 pad 3: BOOT0 -> /SUPER_UART_front_uC/BOOT0
- Q2 pad 1: Net-(Q2-Pad1) -> /SUPER_UART_front_UART1/I2C_PU_EN_B_VCCA
- Q2 pad 2: VDD -> VDD1
- Q3 pad 1: Net-(Q2-Pad1) -> /~RXD_B_OC 
- Q3 pad 2: VDD -> GND
- Q3 pad 3: Net-(Q3-Pad3) -> /~CTS_B_OC 
- Q4 pad 1: Net-(C37-Pad1) -> /SUPER_UART_front_UART1/I2C_PU_EN_B_VCCA
- Q4 pad 2: GND -> VDD1
- Q4 pad 3: Net-(C51-Pad1) -> Net-(Q4-Pad3)
- R1 pad 1: Net-(D48-Pad2) -> /SUPER_UART_front_uC/LED5uC
- R1 pad 2: +3V3 -> /SUPER_UART_front_uC/LED5
- R10 pad 1: (no net) -> /SUPER_UART_front_UART1/RXD_B_VDD1
- R10 pad 2: Net-(D11-Pad2) -> Net-(Q2-Pad3)
- R11 pad 1: (no net) -> /SUPER_UART_front_UART1/RI_D_VDD1
- R11 pad 2: Net-(Q2-Pad3) -> Net-(R11-Pad2)
- R12 pad 1: /SUPER_UART_front_UART234/CTS_A_VDD_VDD -> /SUPER_UART_front_UART1/RXD_B_VDD1
- R12 pad 2: Net-(Q3-Pad3) -> Net-(R12-Pad2)
- R13 pad 1: (no net) -> /SUPER_UART_front_RS232/DTR_D1
- R13 pad 2: Net-(R13-Pad2) -> Net-(LED29-Pad1)
- R14 pad 1: Net-(R14-Pad1) -> /SUPER_UART_front_RS232/RTS_D1
- R14 pad 2: (no net) -> Net-(LED30-Pad1)
- R15 pad 1: /SUPER_UART_front_UART1/RI_D_VDDA -> GND
- R15 pad 2: Net-(R15-Pad2) -> /~RXD_B_OC 
- R16 pad 1: Net-(R16-Pad1) -> /SUPER_UART_front_UART1/CTS_B_VDD1
- R16 pad 2: /SUPER_UART_front_UART1/RXD_B_VDDA -> Net-(Q4-Pad3)
- R17 pad 2: /SUPER_UART_front_UART1/CTS_B_VDDA -> /SUPER_UART_front_UART1/CTS_B_VDD1
- R2 pad 1: Net-(D49-Pad2) -> GND
- R2 pad 2: +3V3 -> /SUPER_UART_front_uC/BOOT0
- R3 pad 1: ISO_GND -> Net-(LED21-Pad2)
- R3 pad 2: BOOT0 -> +3V3
- R4 pad 1: Net-(D48-Pad1) -> /SUPER_UART_front_RS232/DTR_FORCE
- R5 pad 1: PWREN -> Net-(LED22-Pad2)
- R6 pad 1: Net-(D49-Pad1) -> /SUPER_UART_front_RS232/RTS_FORCE
- R7 pad 1: /SUPER_UART_front_UART1/DCD_D -> /SUPER_UART_front_UART1/RXD_D_LED
- R8 pad 1: /SUPER_UART_front_UART1/DTR_D -> /SUPER_UART_front_UART1/TXD_D_LED
- R8 pad 2: Net-(D9-Pad1) -> Net-(LED27-Pad2)
- R9 pad 1: (no net) -> Net-(R9-Pad1)
- R9 pad 2: Net-(D10-Pad2) -> /SUPER_UART_front_UART1/DTR_B_VDD1
- RN1 pad 1: /SUPER_UART_front_UART1/TXD_D_VDDA -> /SUPER_UART_front_uC/LED1
- RN1 pad 2: /SUPER_UART_front_UART1/DTR_D_VDDA -> /SUPER_UART_front_uC/LED2
- RN1 pad 3: /SUPER_UART_front_UART1/RTS_D_VDDA -> /SUPER_UART_front_uC/LED3
- RN1 pad 4: (no net) -> /SUPER_UART_front_uC/LED4
- RN1 pad 5: Net-(RN1-Pad5) -> /SUPER_UART_front_uC/LED4uC
- RN1 pad 6: Net-(RN1-Pad6) -> /SUPER_UART_front_uC/LED3uC
- RN1 pad 7: Net-(RN1-Pad7) -> /SUPER_UART_front_uC/LED2uC
- RN1 pad 8: Net-(RN1-Pad8) -> /SUPER_UART_front_uC/LED1uC
- RN2 pad 1: /SUPER_UART_front_UART234/DTR_B_VDD -> /SUPER_UART_front_uC/SW1
- RN2 pad 2: /SUPER_UART_front_UART234/TXD_B_VDD -> /SUPER_UART_front_uC/SW2
- RN2 pad 3: /SUPER_UART_front_UART234/RXD_B_VDD -> /SUPER_UART_front_uC/SW3
- RN2 pad 4: /SUPER_UART_front_UART234/CTS_B_VDD -> /SUPER_UART_front_uC/SW4
- RN2 pad 5: Net-(RN2-Pad5) -> +3V3
- RN2 pad 6: Net-(RN2-Pad6) -> +3V3
- RN2 pad 7: Net-(RN2-Pad7) -> +3V3
- RN2 pad 8: Net-(RN2-Pad8) -> +3V3
- RN3 pad 1: /SUPER_UART_front_UART234/DTR_C_VDD -> Net-(LED23-Pad1)
- RN3 pad 2: /SUPER_UART_front_UART234/TXD_C_VDD -> Net-(LED24-Pad1)
- RN3 pad 3: /SUPER_UART_front_UART234/RXD_C_VDD -> Net-(LED25-Pad1)
- RN3 pad 4: /SUPER_UART_front_UART234/CTS_C_VDD -> Net-(LED26-Pad1)
- RN3 pad 5: Net-(RN3-Pad5) -> /DCD_D 
- RN3 pad 6: Net-(RN3-Pad6) -> /DSR_D 
- RN3 pad 7: Net-(RN3-Pad7) -> /CTS_D 
- RN3 pad 8: Net-(RN3-Pad8) -> /RI_D 
- RN4 pad 1: /SUPER_UART_front_UART234/DTR_D_VDD -> /SUPER_UART_front_UART1/TXD_D_VDD1
- RN4 pad 2: /SUPER_UART_front_UART234/TXD_D_VDD -> /SUPER_UART_front_UART1/DTR_D_VDD1
- RN4 pad 3: /SUPER_UART_front_UART234/RXD_D_VDD -> /SUPER_UART_front_UART1/RTS_D_VDD1
- RN4 pad 4: /SUPER_UART_front_UART234/CTS_D_VDD -> /SUPER_UART_front_UART1/TXD_B_VDD1
- RN5 pad 1: /SUPER_UART_front_UART234/CTS_B -> /SUPER_UART_front_UART1/RXD_D_VDD1
- RN5 pad 2: RXD_B_LED -> /SUPER_UART_front_UART1/CTS_D_VDD1
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Routing:
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
Commit message: Working on schematic
Parts:
- added TP10: Testpoint, pnConnector:TP_1mm, F.Cu at (36.1, 170.5)
- added TP11: Testpoint, pnConnector:TP_1mm, F.Cu at (53.2, 167.0)
- added TP12: Testpoint, pnConnector:TP_1mm, F.Cu at (68.2, 117.2)
- added TP13: Testpoint, pnConnector:TP_1mm, F.Cu at (53.9, 123.0)
- added TP14: Testpoint, pnConnector:TP_1mm, F.Cu at (74.8, 123.0)
- added TP15: Testpoint, pnConnector:TP_1mm, F.Cu at (81.3, 167.3)
- added TP16: Testpoint, pnConnector:TP_1mm, F.Cu at (59.5, 135.7)
- added TP17: Testpoint, pnConnector:TP_1mm, F.Cu at (60.2, 171.8)
- added TP18: Testpoint, pnConnector:TP_1mm, F.Cu at (81.9, 123.0)
- added TP19: Testpoint, pnConnector:TP_1mm, F.Cu at (53.2, 171.6)
- added TP20: Testpoint, pnConnector:TP_1mm, F.Cu at (74.8, 127.6)
- added TP21: Testpoint, pnConnector:TP_1mm, F.Cu at (52.7, 131.1)
- added TP22: Testpoint, pnConnector:TP_1mm, F.Cu at (59.8, 126.5)
- added TP23: Testpoint, pnConnector:TP_1mm, F.Cu at (60.2, 167.2)
- added TP24: Testpoint, pnConnector:TP_1mm, F.Cu at (73.3, 132.2)
- added TP25: Testpoint, pnConnector:TP_1mm, F.Cu at (68.2, 112.6)
- added TP26: Testpoint, pnConnector:TP_1mm, F.Cu at (70.6, 136.8)
- added TP27: Testpoint, pnConnector:TP_1mm, F.Cu at (52.4, 135.7)
- added TP28: Testpoint, pnConnector:TP_1mm, F.Cu at (81.9, 127.6)
- added TP29: Testpoint, pnConnector:TP_1mm, F.Cu at (88.9, 123.0)
- added TP3: Testpoint, pnConnector:TP_1mm, F.Cu at (49.9, 176.2)
- added TP30: Testpoint, pnConnector:TP_1mm, F.Cu at (51.9, 140.3)
- added TP31: Testpoint, pnConnector:TP_1mm, F.Cu at (57.0, 176.4)
- added TP32: Testpoint, pnConnector:TP_1mm, F.Cu at (70.6, 146.0)
- added TP33: Testpoint, pnConnector:TP_1mm, F.Cu at (59.8, 131.1)
- added TP34: Testpoint, pnConnector:TP_1mm, F.Cu at (59.0, 140.3)
- added TP35: Testpoint, pnConnector:TP_1mm, F.Cu at (88.9, 127.6)
- added TP4: Testpoint, pnConnector:TP_1mm, F.Cu at (77.6, 136.8)
- added TP5: Testpoint, pnConnector:TP_1mm, F.Cu at (70.6, 141.4)
- added TP6: Testpoint, pnConnector:TP_1mm, F.Cu at (80.4, 132.2)
- added TP7: Testpoint, pnConnector:TP_1mm, F.Cu at (63.6, 118.3)
- added TP8: Testpoint, pnConnector:TP_1mm, F.Cu at (48.7, 148.3)
- added TP9: Testpoint, pnConnector:TP_1mm, F.Cu at (42.9, 175.3)
- C1, C10, C11, C12, C13, C14, C15, C16, C17, C18, C19, C2, C20, C21, C22, C23, C24, C25, C26, C27, C28, C29, C3, C30, C31, C32, C33, C34, C35, C36, C37, C38, C39, C4, C40, C41, C42, C43, C44, C45, C46, C47, C5, C6, C7, C8, C9, CON1, CON2, CON3, D1, D10, D11, D12, D13, D2, D3, D4, D5, D6, D7, D8, D9, MH1, MH2, Q1, Q10, Q11, Q2, Q3, Q4, Q5, Q6, Q7, Q8, Q9, R1, R10, R11, R12, R13, R14, R15, R16, R17, R18, R19, R2, R20, R21, R22, R23, R24, R25, R26, R27, R28, R29, R3, R30, R31, R32, R33, R34, R35, R36, R37, R38, R39, R4, R40, R41, R42, R43, R44, R5, R6, R7, R8, R9, RN1, RN2, RN3, RN4, RN5, RN7, RN8, RN9, SW1, SW10, SW11, SW12, SW13, SW14, SW15, SW16, SW17, SW18, SW19, SW2, SW3, SW4, SW5, SW6, SW7, SW8, SW9, TP1, TP2, U1, U10, U11, U12, U13, U14, U2, U3, U4, U5, U6, U7, U8, U9: moved to F.Cu
- CON4, CON5: value UART A -> PORT D; moved to F.Cu
- CON6: value UART D -> PORT B; moved to F.Cu
- CON7: value UART B -> PORT A; moved to F.Cu
- CON8: value UART C -> PORT C
- LED1, LED10, LED11, LED12, LED13, LED14, LED15, LED16, LED17, LED18, LED19, LED2, LED20, LED21, LED22, LED3, LED4, LED5, LED6, LED7, LED8, LED9: footprint pnSemiconductor:LED_3.2x2 -> pnSemiconductor:0805D; moved to F.Cu
- LED23, LED24, LED25, LED26, LED27, LED28, LED29, LED30, LED31, LED32, LED33, LED34, LED35, LED36, LED37, LED38: footprint pnSemiconductor:LED0603_R -> pnSemiconductor:0805D; moved to F.Cu
- LED39, LED40, LED41, LED42: footprint pnSemiconductor:LED0603_R -> pnSemiconductor:0805D
- moved CON1 187.5 mm to (228.3, 116.7)
- moved D1 180.5 mm to (21.0, 163.6), turned to 90 degrees
- moved LED11 173.6 mm to (34.0, 22.4)
- moved C4 172.4 mm to (39.8, 159.0), turned to 270 degrees
- moved LED10 172.1 mm to (24.5, 36.1)
- moved LED14 171.0 mm to (24.5, 43.4)
- moved LED12 169.2 mm to (24.5, 22.4)
- moved C11 164.9 mm to (28.9, 90.5), turned to 180 degrees
- moved Q5 161.7 mm to (172.3, 63.9)
- moved LED9 159.0 mm to (34.0, 36.1)
- moved LED26 156.2 mm to (74.0, 43.0), turned to 90 degrees
- moved LED13 156.1 mm to (24.5, 57.1)
- moved SW14 156.1 mm to (24.5, 47.4), turned to 270 degrees
- moved SW10 155.7 mm to (24.5, 32.1), turned to 90 degrees
- moved LED37 155.4 mm to (38.0, 47.2)
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Connections:
- net /~CTS_A_OC  renamed /~CTS_A_OC
- net /~CTS_B_OC  renamed /~CTS_B_OC
- net /~RXD_A_OC  renamed /~RXD_A_OC
- net /~RXD_B_OC  renamed /~RXD_B_OC
- TP1 pad 1: Net-(TP1-Pad1) -> /SUPER_UART_front_RS232/RXD_D3
- TP2 pad 1: Net-(TP2-Pad1) -> /TXD_D 
- U12 pad 24: (no net) -> VDD2
- U8 pad 10: Net-(TP2-Pad1) -> (no net)
- U8 pad 9: Net-(TP1-Pad1) -> (no net)
Other:
- board size 100 x 35 mm -> 100 x 43 mm

Commit message: PCB placement
Parts:
- removed CON1: PIN-2x20, PIN-2x20_N
- removed U3: AP7333-33SAG-7, SOT23-3_N
- added Q12: PDTA143ZT, niceSemiconductors:SOT23-3_N, B.Cu at (90.6, 45.0)
- added Q13: N-MOS_small, SOT23-3_N, B.Cu at (39.8, 6.80)
- added Q14: N-MOS_small, SOT23-3_N, B.Cu at (58.9, 5.60)
- added R48: 10k, 0603_R_N, B.Cu at (93.3, 42.4)
- C1, C10, C11, C12, C13, C14, C15, C16, C17, C18, C19, C2, C20, C21, C22, C23, C24, C25, C26, C27, C28, C29, C3, C30, C31, C32, C33, C34, C35, C36, C37, C38, C39, C4, C40, C41, C42, C43, C44, C45, C46, C47, C48, C5, C6, C7, C8, C9, CON2, D1, D10, D11, D12, D13, D2, D3, D4, D5, D6, D7, D8, D9, Q1, Q10, Q11, Q2, Q4, Q5, Q6, Q7, Q9, R10, R11, R12, R13, R14, R15, R16, R17, R18, R19, R2, R20, R21, R22, R23, R24, R25, R26, R27, R28, R29, R3, R30, R31, R32, R33, R34, R35, R36, R37, R38, R39, R4, R40, R41, R42, R43, R44, R45, R46, R47, R5, R6, R7, R8, R9, TP1, TP10, TP11, TP12, TP13, TP14, TP15, TP16, TP17, TP18, TP19, TP2, TP20, TP21, TP22, TP23, TP24, TP25, TP26, TP27, TP28, TP29, TP3, TP30, TP31, TP32, TP33, TP34, TP35, TP4, TP5, TP6, TP7, TP8, TP9, U1, U10, U11, U12, U13, U14, U15, U16, U2, U4, U5, U6, U7, U8, U9: moved to B.Cu
- Q3, Q8: value 2N7002PS -> N-MOS_small; footprint niceSemiconductors:SC70-6_N -> SOT23-3_N; moved to B.Cu
- R1: footprint pnRLC:0805_JUMPER -> niceRLC:0603_R_N; moved to B.Cu
- RN1, RN2, RN3, RN4, RN5, RN6, RN7, RN9: footprint pnRLC:4x0603_N -> niceRLC:4x0603_N; moved to B.Cu
- RN8: footprint 4x0603_N -> niceRLC:4x0603_N; moved to B.Cu
- moved R35 177.3 mm to (33.5, 5.00)
- moved R32 174.9 mm to (36.5, 7.80), turned to 180 degrees
- moved R33 173.8 mm to (36.5, 6.20)
- moved R34 169.3 mm to (40.0, 9.40)
- moved C39 163.9 mm to (32.5, 10.1), turned to 270 degrees
- moved C40 161.9 mm to (34.1, 10.1), turned to 270 degrees
- moved R39 161.8 mm to (55.6, 5.00)
- moved R36 159.4 mm to (55.6, 6.60), turned to 180 degrees
- moved Q7 157.8 mm to (36.7, 10.4), turned to 180 degrees
- moved U14 157.7 mm to (33.3, 7.20), turned to 90 degrees
- moved C45 155.8 mm to (51.6, 8.90), turned to 270 degrees
- moved R41 155.7 mm to (59.1, 8.20)
- moved C46 155.3 mm to (53.2, 8.90), turned to 270 degrees
- moved U15 150.6 mm to (52.4, 6.00), turned to 90 degrees
- moved Q9 145.2 mm to (55.8, 9.20), turned to 180 degrees
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Connections:
- net /SUPER_UART_front_UART1/~VDD1_EN renamed /SUPER_UART_front_RS232/~VDD1_EN
- Q10 pad 1: /SUPER_UART_front_UART234/VDD2_SEL1 -> /SUPER_UART_front_UART234/VDD2_SEL3
- Q10 pad 6: Net-(C48-Pad1) -> Net-(Q10-Pad6)
- Q11 pad 1: /SUPER_UART_front_UART234/VDD2_SEL3 -> /SUPER_UART_front_UART234/VDD2_SEL1
- Q11 pad 3: Net-(Q11-Pad3) -> Net-(C48-Pad1)
- Q3 pad 3: /~CTS_B_OC -> /SUPER_UART_front_UART1/RXD_B_VDD1
- Q5 pad 1: /SUPER_UART_front_UART1/VDD1_SEL1 -> /SUPER_UART_front_UART1/VDD1_SEL3
- Q5 pad 6: Net-(C32-Pad1) -> Net-(Q5-Pad6)
- Q6 pad 1: /SUPER_UART_front_UART1/VDD1_SEL3 -> /SUPER_UART_front_UART1/VDD1_SEL1
- Q6 pad 3: Net-(Q6-Pad3) -> Net-(C32-Pad1)
- Q8 pad 1: /~CTS_A_OC -> /~CTS_B_OC
- Q8 pad 3: /~RXD_A_OC -> /SUPER_UART_front_UART1/CTS_B_VDD1
- R25 pad 1: Net-(Q6-Pad3) -> Net-(Q5-Pad6)
- R44 pad 1: Net-(Q11-Pad3) -> Net-(Q10-Pad6)
- RN4 pad 1: /SUPER_UART_front_UART1/TXD_D_VDD1 -> /SUPER_UART_front_UART1/TXD_B_VDD1
- RN4 pad 2: /SUPER_UART_front_UART1/DTR_D_VDD1 -> /SUPER_UART_front_UART1/RTS_D_VDD1
- RN4 pad 3: /SUPER_UART_front_UART1/RTS_D_VDD1 -> /SUPER_UART_front_UART1/DTR_D_VDD1
- RN4 pad 4: /SUPER_UART_front_UART1/TXD_B_VDD1 -> /SUPER_UART_front_UART1/TXD_D_VDD1
- RN5 pad 1: /SUPER_UART_front_UART1/RXD_D_VDD1 -> /SUPER_UART_front_UART1/DSR_D_VDD1
- RN5 pad 2: /SUPER_UART_front_UART1/CTS_D_VDD1 -> /SUPER_UART_front_UART1/DCD_D_VDD1
- RN5 pad 3: /SUPER_UART_front_UART1/DCD_D_VDD1 -> /SUPER_UART_front_UART1/CTS_D_VDD1
- RN5 pad 4: /SUPER_UART_front_UART1/DSR_D_VDD1 -> /SUPER_UART_front_UART1/RXD_D_VDD1
- RN7 pad 1: /SUPER_UART_front_UART234/TXD_A_VDD2 -> /SUPER_UART_front_UART234/DTR_C_VDD2
- RN7 pad 2: /SUPER_UART_front_UART234/DTR_A_VDD2 -> /SUPER_UART_front_UART234/TXD_C_VDD2
- RN7 pad 3: /SUPER_UART_front_UART234/TXD_C_VDD2 -> /SUPER_UART_front_UART234/DTR_A_VDD2
- RN7 pad 4: /SUPER_UART_front_UART234/DTR_C_VDD2 -> /SUPER_UART_front_UART234/TXD_A_VDD2
- U12 pad 18: Net-(RN7-Pad5) -> Net-(RN7-Pad8)
- U12 pad 19: Net-(RN7-Pad6) -> Net-(RN7-Pad7)
- U12 pad 20: Net-(RN7-Pad7) -> Net-(RN7-Pad6)
- U12 pad 21: Net-(RN7-Pad8) -> Net-(RN7-Pad5)
- U5 pad 22: +3V3 -> Net-(Q12-Pad3)
- U7 pad 18: Net-(RN4-Pad5) -> Net-(RN4-Pad8)
- U7 pad 19: Net-(RN4-Pad6) -> Net-(RN4-Pad7)
- U7 pad 20: Net-(RN4-Pad7) -> Net-(RN4-Pad6)
- U7 pad 21: Net-(RN4-Pad8) -> Net-(RN4-Pad5)
- U8 pad 18: Net-(RN5-Pad5) -> Net-(RN5-Pad8)
- U8 pad 19: Net-(RN5-Pad6) -> Net-(RN5-Pad7)
- U8 pad 20: Net-(RN5-Pad7) -> Net-(RN5-Pad6)
- U8 pad 21: Net-(RN5-Pad8) -> Net-(RN5-Pad5)
Routing:
- net Net-(Q12-Pad3): track 0.00 -> 7.68 mm
- net GND: track 0.00 -> 6.27 mm, vias 0 -> 2
- net Net-(C12-Pad2): track 0.00 -> 5.76 mm
- net +3V3: track 0.00 -> 5.14 mm, vias 0 -> 2
- net Net-(C15-Pad1): track 0.00 -> 4.50 mm
- net Net-(C14-Pad2): track 0.00 -> 3.78 mm
- net Net-(C16-Pad1): track 0.00 -> 2.23 mm
- net Net-(C12-Pad1): track 0.00 -> 2.20 mm
- net Net-(C14-Pad1): track 0.00 -> 2.17 mm
