File: kicad/front/SUPER_UART_front_RS232.sch (KiCad schematic (older format))
At the start: 21 parts, among them CON5 RS232, SW16 DTR, SW17 RTS, U4 74HC08P, U5 MAX3243EIPW, U7 74HC08P

Commit message: Working on schematic
Parts:
- removed C21, C23: 470n, 0603_N, symbol C
- added C14, C16: 1u, 0603_N, symbol C
- added LED23: RI, pnSemiconductor:LED0603_R, symbol diode_LED
- added LED24: CTS, pnSemiconductor:LED0603_R, symbol diode_LED
- added LED25: DSR, pnSemiconductor:LED0603_R, symbol diode_LED
- added LED26: DCD, pnSemiconductor:LED0603_R, symbol diode_LED
- added RN3: R, pnRLC:4x0603_N, symbol R_network_4
- C13: renamed from C16; value 100n -> 1u; Fieldname (none) -> Value
- C15: renamed from C22; value 470n -> 1u; Fieldname (none) -> Value
- renumbered C4 to C12, C24 to C17, C25 to C18, CON5 to CON3, D48 to LED21, D49 to LED22, R1 to R3, R2 to R4, R4 to R5, SW16 to SW18, SW17 to SW19, U7 to U6
Connections:
- net +3V3: now also LED23.2 (C), LED24.2 (C), LED25.2 (C), LED26.2 (C)
- net CTS_D: now also RN3.7
- net DCD_D: now also RN3.5
- net DSR_D: now also RN3.6
- net GND: now also C16.2
- net RI_D: now also RN3.8
- net at U5.1 (C2+): now also C14.1
- net at U5.2 (C2-): now also C14.2
- net at U5.27 (V+): now also C16.1
- new net: LED24.1 (A), RN3.2
- new net: LED23.1 (A), RN3.1
- new net: LED25.1 (A), RN3.3
- new net: LED26.1 (A), RN3.4
Other:
- moved on the sheet: C17, C18, U4E, U6E

Commit message: Working on schematic
Parts:
- LED21, LED22: footprint pnSemiconductor:LED_3.2x2 -> pnSemiconductor:0805D
- LED23, LED24, LED25, LED26: footprint pnSemiconductor:LED0603_R -> pnSemiconductor:0805D
Changed lines of the file:
@@
 $EndComp
 $Comp
-L GND #PWR029
+L GND #PWR035
 U 1 1 5933AA2F
 P 5550 2900
-F 0 "#PWR029" H 5580 2870 10  0001 C CNN
+F 0 "#PWR035" H 5580 2870 10  0001 C CNN
 F 1 "GND" H 5550 2775 40  0001 C CNN
 F 2 "" H 5550 2900 50  0001 C CNN
@@
 $EndComp
 $Comp
-L +3V3 #PWR030
+L +3V3 #PWR036
 U 1 1 5933AA35
 P 5550 2500
-F 0 "#PWR030" H 5580 2530 10  0001 C CNN
+F 0 "#PWR036" H 5580 2530 10  0001 C CNN
 F 1 "+3V3" H 5550 2630 50  0000 C CNN
 F 2 "" H 5550 2500 50  0001 C CNN
@@
 $EndComp
 $Comp
-L GND #PWR031
+L GND #PWR037
 U 1 1 5933AA3B
 P 5550 3800
-F 0 "#PWR031" H 5580 3770 10  0001 C CNN
+F 0 "#PWR037" H 5580 3770 10  0001 C CNN
 F 1 "GND" H 5550 3675 40  0001 C CNN
 F 2 "" H 5550 3800 50  0001 C CNN
@@
 NoConn ~ 5900 3250
 $Comp
-L GND #PWR032
+L GND #PWR038
 U 1 1 5933AA42
 P 8050 3800
-F 0 "#PWR032" H 8080 3770 10  0001 C CNN
+F 0 "#PWR038" H 8080 3770 10  0001 C CNN
 F 1 "GND" H 8050 3675 40  0001 C CNN
 F 2 "" H 8050 3800 50  0001 C CNN
@@
 $EndComp
 $Comp
-L GND #PWR033
+L GND #PWR039
 U 1 1 5933AA67
 P 10600 3250
-F 0 "#PWR033" H 10630 3220 10  0001 C CNN
+F 0 "#PWR039" H 10630 3220 10  0001 C CNN
 F 1 "GND" H 10600 3125 40  0001 C CNN
 F 2 "" H 10600 3250 50  0001 C CNN
@@
 $EndComp
 $Comp
-L GND #PWR034
+L GND #PWR040
 U 1 1 5933AA74
 P 9950 3250
-F 0 "#PWR034" H 9980 3220 10  0001 C CNN
+F 0 "#PWR040" H 9980 3220 10  0001 C CNN
 F 1 "GND" H 9950 3125 40  0001 C CNN
 F 2 "" H 9950 3250 50  0001 C CNN
@@
 DTR_232
 $Comp
-L GND #PWR035
+L GND #PWR041
 U 1 1 5933AA89
 P 10300 2550
-F 0 "#PWR035" H 10330 2520 10  0001 C CNN
+F 0 "#PWR041" H 10330 2520 10  0001 C CNN
 F 1 "GND" H 10300 2425 40  0001 C CNN
 F 2 "" H 10300 2550 50  0001 C CNN
@@
 F 0 "LED21" H 1725 1510 60  0000 L CNN
 F 1 "DTR" H 1725 1410 40  0000 L CNN
-F 2 "pnSemiconductor:LED_3.2x2" H 1725 1350 40  0001 L CNN
+F 2 "pnSemiconductor:0805D" H 1725 1350 40  0001 L CNN
 F 3 "" H 1650 1450 60  0001 C CNN
 	1    1650 1450
@@
 F 0 "LED22" H 1725 3160 60  0000 L CNN
 F 1 "RTS" H 1725 3060 40  0000 L CNN
-F 2 "pnSemiconductor:LED_3.2x2" H 1725 3000 40  0001 L CNN
+F 2 "pnSemiconductor:0805D" H 1725 3000 40  0001 L CNN
 F 3 "" H 1650 3100 60  0001 C CNN
 	1    1650 3100
@@
 $EndComp
 $Comp
-L GND #PWR036
+L GND #PWR042
 U 1 1 5933BD74
 P 1650 2250
-F 0 "#PWR036" H 1650 2050 50  0001 C CNN
+F 0 "#PWR042" H 1650 2050 50  0001 C CNN
 F 1 "GND" H 1650 2125 30  0001 C CNN
 F 2 "" H 1650 2250 50  0001 C CNN
@@
 $EndComp
 $Comp
-L +3V3 #PWR037
+L +3V3 #PWR043
 U 1 1 5933BD81
 P 1650 1050
-F 0 "#PWR037" H 1680 1080 10  0001 C CNN
+F 0 "#PWR043" H 1680 1080 10  0001 C CNN
 F 1 "+3V3" H 1650 1180 50  0000 C CNN
 F 2 "" H 1650 1050 50  0001 C CNN
@@
 $EndComp
 $Comp
-L GND #PWR038
+L GND #PWR044
 U 1 1 5933BD88
 P 1650 3800
-F 0 "#PWR038" H 1650 3600 50  0001 C CNN
+F 0 "#PWR044" H 1650 3600 50  0001 C CNN
 F 1 "GND" H 1650 3675 30  0001 C CNN
 F 2 "" H 1650 3800 50  0001 C CNN
@@
 $EndComp
 $Comp
-L +3V3 #PWR039
+L +3V3 #PWR045
 U 1 1 5933BD95
 P 1650 2700
-F 0 "#PWR039" H 1680 2730 10  0001 C CNN
+F 0 "#PWR045" H 1680 2730 10  0001 C CNN
 F 1 "+3V3" H 1650 2830 50  0000 C CNN
 F 2 "" H 1650 2700 50  0001 C CNN
@@
 $EndComp
 $Comp
-L +3V3 #PWR040
+L +3V3 #PWR046
 U 1 1 5933BDC9
 P 2250 2700
-F 0 "#PWR040" H 2280 2730 10  0001 C CNN
+F 0 "#PWR046" H 2280 2730 10  0001 C CNN
 F 1 "+3V3" H 2250 2830 50  0000 C CNN
 F 2 "" H 2250 2700 50  0001 C CNN
@@
 $EndComp
 $Comp
-L +3V3 #PWR041
+L +3V3 #PWR047
 U 1 1 5933BDD9
 P 2250 1050
-F 0 "#PWR041" H 2280 1080 10  0001 C CNN
+F 0 "#PWR047" H 2280 1080 10  0001 C CNN
 F 1 "+3V3" H 2250 1180 50  0000 C CNN
 F 2 "" H 2250 1050 50  0001 C CNN
@@
 	1650 1800 2450 1800
 $Comp
-L +3V3 #PWR042
+L +3V3 #PWR048
 U 1 1 5933BDE3
 P 2100 6700
-F 0 "#PWR042" H 2130 6730 10  0001 C CNN
+F 0 "#PWR048" H 2130 6730 10  0001 C CNN
 F 1 "+3V3" H 2100 6830 50  0000 C CNN
 F 2 "" H 2100 6700 50  0001 C CNN
@@
 $EndComp
 $Comp
-L GND #PWR043
+L GND #PWR049
 U 1 1 5933BDE9
 P 2100 7300
-F 0 "#PWR043" H 2100 7100 50  0001 C CNN
+F 0 "#PWR049" H 2100 7100 50  0001 C CNN
 F 1 "GND" H 2100 7175 30  0001 C CNN
 F 2 "" H 2100 7300 50  0001 C CNN
@@
 $EndComp
 $Comp
-L GND #PWR044
+L GND #PWR050
 U 1 1 5933BDF6
 P 1750 7300
-F 0 "#PWR044" H 1750 7100 50  0001 C CNN
+F 0 "#PWR050" H 1750 7100 50  0001 C CNN
 F 1 "GND" H 1750 7175 30  0001 C CNN
 F 2 "" H 1750 7300 50  0001 C CNN
@@
 $EndComp
 $Comp
-L +3V3 #PWR045
+L +3V3 #PWR051
 U 1 1 5933BDFC
 P 1750 6700
-F 0 "#PWR045" H 1780 6730 10  0001 C CNN
+F 0 "#PWR051" H 1780 6730 10  0001 C CNN
 F 1 "+3V3" H 1750 6830 50  0000 C CNN
 F 2 "" H 1750 6700 50  0001 C CNN
@@
 	2100 6750 2100 6700
 $Comp
-L +3V3 #PWR046
+L +3V3 #PWR052
 U 1 1 5933BE06
 P 3000 6700
-F 0 "#PWR046" H 3030 6730 10  0001 C CNN
+F 0 "#PWR052" H 3030 6730 10  0001 C CNN
 F 1 "+3V3" H 3000 6830 50  0000 C CNN
 F 2 "" H 3000 6700 50  0001 C CNN
@@
 $EndComp
 $Comp
-L GND #PWR047
+L GND #PWR053
 U 1 1 5933BE0C
 P 3000 7300
-F 0 "#PWR047" H 3000 7100 50  0001 C CNN
+F 0 "#PWR053" H 3000 7100 50  0001 C CNN
 F 1 "GND" H 3000 7175 30  0001 C CNN
 F 2 "" H 3000 7300 50  0001 C CNN
@@
 $EndComp
 $Comp
-L GND #PWR048
+L GND #PWR054
 U 1 1 5933BE19
 P 2650 7300
-F 0 "#PWR048" H 2650 7100 50  0001 C CNN
+F 0 "#PWR054" H 2650 7100 50  0001 C CNN
 F 1 "GND" H 2650 7175 30  0001 C CNN
 F 2 "" H 2650 7300 50  0001 C CNN
@@
 $EndComp
 $Comp
-L +3V3 #PWR049
+L +3V3 #PWR055
 U 1 1 5933BE1F
 P 2650 6700
-F 0 "#PWR049" H 2680 6730 10  0001 C CNN
+F 0 "#PWR055" H 2680 6730 10  0001 C CNN
 F 1 "+3V3" H 2650 6830 50  0000 C CNN
 F 2 "" H 2650 6700 50  0001 C CNN
@@
 F 0 "LED24" H 6175 5310 60  0000 L CNN
 F 1 "CTS" H 6175 5210 40  0000 L CNN
-F 2 "pnSemiconductor:LED0603_R" H 6175 5150 40  0001 L CNN
+F 2 "pnSemiconductor:0805D" H 6175 5150 40  0001 L CNN
 F 3 "" H 6100 5250 60  0001 C CNN
 	1    6100 5250
@@
 F 0 "LED23" H 5775 5310 60  0000 L CNN
 F 1 "RI" H 5775 5210 40  0000 L CNN
-F 2 "pnSemiconductor:LED0603_R" H 5775 5150 40  0001 L CNN
+F 2 "pnSemiconductor:0805D" H 5775 5150 40  0001 L CNN
 F 3 "" H 5700 5250 60  0001 C CNN
 	1    5700 5250
@@
 $EndComp
 $Comp
-L +3V3 #PWR050
+L +3V3 #PWR056
 U 1 1 5943325E
 P 6100 5100
-F 0 "#PWR050" H 6130 5130 10  0001 C CNN
+F 0 "#PWR056" H 6130 5130 10  0001 C CNN
 F 1 "+3V3" H 6100 5230 50  0000 C CNN
 F 2 "" H 6100 5100 50  0001 C CNN
@@
 $EndComp
 $Comp
-L +3V3 #PWR051
+L +3V3 #PWR057
 U 1 1 59433264
 P 5700 5100
-F 0 "#PWR051" H 5730 5130 10  0001 C CNN
+F 0 "#PWR057" H 5730 5130 10  0001 C CNN
 F 1 "+3V3" H 5700 5230 50  0000 C CNN
 F 2 "" H 5700 5100 50  0001 C CNN
@@
 	4850 6600 5250 6600
 $Comp
-L +3V3 #PWR052
+L +3V3 #PWR058
 U 1 1 59433291
 P 6100 5950
-F 0 "#PWR052" H 6130 5980 10  0001 C CNN
+F 0 "#PWR058" H 6130 5980 10  0001 C CNN
 F 1 "+3V3" H 6100 6080 50  0000 C CNN
 F 2 "" H 6100 5950 50  0001 C CNN
@@
 $EndComp
 $Comp
-L +3V3 #PWR053
+L +3V3 #PWR059
 U 1 1 59433297
 P 5600 6000
-F 0 "#PWR053" H 5630 6030 10  0001 C CNN
+F 0 "#PWR059" H 5630 6030 10  0001 C CNN
 F 1 "+3V3" H 5600 6130 50  0000 C CNN
 F 2 "" H 5600 6000 50  0001 C CNN
@@
 F 0 "LED26" H 5675 6210 60  0000 L CNN
 F 1 "DCD" H 5675 6110 40  0000 L CNN
-F 2 "pnSemiconductor:LED0603_R" H 5675 6050 40  0001 L CNN
+F 2 "pnSemiconductor:0805D" H 5675 6050 40  0001 L CNN
 F 3 "" H 5600 6150 60  0001 C CNN
 	1    5600 6150
@@
 F 0 "LED25" H 6175 6160 60  0000 L CNN
 F 1 "DSR" H 6175 6060 40  0000 L CNN
-F 2 "pnSemiconductor:LED0603_R" H 6175 6000 40  0001 L CNN
+F 2 "pnSemiconductor:0805D" H 6175 6000 40  0001 L CNN
 F 3 "" H 6100 6100 60  0001 C CNN
 	1    6100 6100

Commit message: PCB placement
Parts:
- added Q12: PDTA143ZT, niceSemiconductors:SOT23-3_N, symbol PDTA143ZT
- added R48: 10k, 0603_R_N, symbol R_V
- RN3: footprint pnRLC:4x0603_N -> niceRLC:4x0603_N
Connections:
- net +3V3: now also Q12.2 (E); no longer U5.22 (~FORCEOFF)
- net GND: now also R48.1
- new net: Q12.3 (C), R48.2, U5.22 (~FORCEOFF)
- new net ~VDD1_EN: Q12.1 (B)
Changed lines of the file:
@@
 $EndComp
 $Comp
-L GND #PWR035
+L GND #PWR032
 U 1 1 5933AA2F
 P 5550 2900
-F 0 "#PWR035" H 5580 2870 10  0001 C CNN
+F 0 "#PWR032" H 5580 2870 10  0001 C CNN
 F 1 "GND" H 5550 2775 40  0001 C CNN
 F 2 "" H 5550 2900 50  0001 C CNN
@@
 $EndComp
 $Comp
-L +3V3 #PWR036
+L +3V3 #PWR033
 U 1 1 5933AA35
 P 5550 2500
-F 0 "#PWR036" H 5580 2530 10  0001 C CNN
+F 0 "#PWR033" H 5580 2530 10  0001 C CNN
 F 1 "+3V3" H 5550 2630 50  0000 C CNN
 F 2 "" H 5550 2500 50  0001 C CNN
@@
 $EndComp
 $Comp
-L GND #PWR037
+L GND #PWR034
 U 1 1 5933AA3B
 P 5550 3800
-F 0 "#PWR037" H 5580 3770 10  0001 C CNN
+F 0 "#PWR034" H 5580 3770 10  0001 C CNN
 F 1 "GND" H 5550 3675 40  0001 C CNN
 F 2 "" H 5550 3800 50  0001 C CNN
@@
 NoConn ~ 5900 3250
 $Comp
-L GND #PWR038
+L GND #PWR035
 U 1 1 5933AA42
 P 8050 3800
-F 0 "#PWR038" H 8080 3770 10  0001 C CNN
+F 0 "#PWR035" H 8080 3770 10  0001 C CNN
 F 1 "GND" H 8050 3675 40  0001 C CNN
 F 2 "" H 8050 3800 50  0001 C CNN
@@
 $EndComp
 $Comp
-L GND #PWR039
+L GND #PWR036
 U 1 1 5933AA67
 P 10600 3250
-F 0 "#PWR039" H 10630 3220 10  0001 C CNN
+F 0 "#PWR036" H 10630 3220 10  0001 C CNN
 F 1 "GND" H 10600 3125 40  0001 C CNN
 F 2 "" H 10600 3250 50  0001 C CNN
@@
 $EndComp
 $Comp
-L GND #PWR040
+L GND #PWR037
 U 1 1 5933AA74
 P 9950 3250
-F 0 "#PWR040" H 9980 3220 10  0001 C CNN
+F 0 "#PWR037" H 9980 3220 10  0001 C CNN
 F 1 "GND" H 9950 3125 40  0001 C CNN
 F 2 "" H 9950 3250 50  0001 C CNN
@@
 DTR_232
 $Comp
-L GND #PWR041
+L GND #PWR038
 U 1 1 5933AA89
 P 10300 2550
-F 0 "#PWR041" H 10330 2520 10  0001 C CNN
+F 0 "#PWR038" H 10330 2520 10  0001 C CNN
 F 1 "GND" H 10300 2425 40  0001 C CNN
 F 2 "" H 10300 2550 50  0001 C CNN
@@
 	5550 2800 5550 2900
 Wire Wire Line
-	5800 3150 5900 3150
-Wire Wire Line
-	5800 2550 5800 3150
+	4900 3150 5900 3150
 Wire Wire Line
 	5550 2550 5900 2550
@@
 Wire Wire Line
 	5900 3050 5800 3050
-Connection ~ 5800 3050
 Wire Wire Line
 	5900 2850 5550 2850
@@
 $EndComp
 $Comp
-L GND #PWR042
+L GND #PWR039
 U 1 1 5933BD74
 P 1650 2250
-F 0 "#PWR042" H 1650 2050 50  0001 C CNN
+F 0 "#PWR039" H 1650 2050 50  0001 C CNN
 F 1 "GND" H 1650 2125 30  0001 C CNN
 F 2 "" H 1650 2250 50  0001 C CNN
@@
 $EndComp
 $Comp
-L +3V3 #PWR043
+L +3V3 #PWR040
 U 1 1 5933BD81
 P 1650 1050
-F 0 "#PWR043" H 1680 1080 10  0001 C CNN
+F 0 "#PWR040" H 1680 1080 10  0001 C CNN
 F 1 "+3V3" H 1650 1180 50  0000 C CNN
 F 2 "" H 1650 1050 50  0001 C CNN
@@
 $EndComp
 $Comp
-L GND #PWR044
+L GND #PWR041
 U 1 1 5933BD88
 P 1650 3800
-F 0 "#PWR044" H 1650 3600 50  0001 C CNN
+F 0 "#PWR041" H 1650 3600 50  0001 C CNN
 F 1 "GND" H 1650 3675 30  0001 C CNN
 F 2 "" H 1650 3800 50  0001 C CNN
@@
 $EndComp
 $Comp
-L +3V3 #PWR045
+L +3V3 #PWR042
 U 1 1 5933BD95
 P 1650 2700
-F 0 "#PWR045" H 1680 2730 10  0001 C CNN
+F 0 "#PWR042" H 1680 2730 10  0001 C CNN
 F 1 "+3V3" H 1650 2830 50  0000 C CNN
 F 2 "" H 1650 2700 50  0001 C CNN
@@
 $EndComp
 $Comp
-L +3V3 #PWR046
+L +3V3 #PWR043
 U 1 1 5933BDC9
 P 2250 2700
-F 0 "#PWR046" H 2280 2730 10  0001 C CNN
+F 0 "#PWR043" H 2280 2730 10  0001 C CNN
 F 1 "+3V3" H 2250 2830 50  0000 C CNN
 F 2 "" H 2250 2700 50  0001 C CNN
@@
 $EndComp
 $Comp
-L +3V3 #PWR047
+L +3V3 #PWR044
 U 1 1 5933BDD9
 P 2250 1050
-F 0 "#PWR047" H 2280 1080 10  0001 C CNN
+F 0 "#PWR044" H 2280 1080 10  0001 C CNN
 F 1 "+3V3" H 2250 1180 50  0000 C CNN
 F 2 "" H 2250 1050 50  0001 C CNN
@@
 	1650 1800 2450 1800
 $Comp
-L +3V3 #PWR048
+L +3V3 #PWR045
 U 1 1 5933BDE3
 P 2100 6700
-F 0 "#PWR048" H 2130 6730 10  0001 C CNN
+F 0 "#PWR045" H 2130 6730 10  0001 C CNN
 F 1 "+3V3" H 2100 6830 50  0000 C CNN
 F 2 "" H 2100 6700 50  0001 C CNN
@@
 $EndComp
 $Comp
-L GND #PWR049
+L GND #PWR046
 U 1 1 5933BDE9
 P 2100 7300
-F 0 "#PWR049" H 2100 7100 50  0001 C CNN
+F 0 "#PWR046" H 2100 7100 50  0001 C CNN
 F 1 "GND" H 2100 7175 30  0001 C CNN
 F 2 "" H 2100 7300 50  0001 C CNN
@@
 $EndComp
 $Comp
-L GND #PWR050
+L GND #PWR047
 U 1 1 5933BDF6
 P 1750 7300
-F 0 "#PWR050" H 1750 7100 50  0001 C CNN
+F 0 "#PWR047" H 1750 7100 50  0001 C CNN
 F 1 "GND" H 1750 7175 30  0001 C CNN
 F 2 "" H 1750 7300 50  0001 C CNN
@@
 $EndComp
 $Comp
-L +3V3 #PWR051
+L +3V3 #PWR048
 U 1 1 5933BDFC
 P 1750 6700
-F 0 "#PWR051" H 1780 6730 10  0001 C CNN
+F 0 "#PWR048" H 1780 6730 10  0001 C CNN
 F 1 "+3V3" H 1750 6830 50  0000 C CNN
 F 2 "" H 1750 6700 50  0001 C CNN
@@
 	2100 6750 2100 6700
 $Comp
-L +3V3 #PWR052
+L +3V3 #PWR049
 U 1 1 5933BE06
 P 3000 6700
-F 0 "#PWR052" H 3030 6730 10  0001 C CNN
+F 0 "#PWR049" H 3030 6730 10  0001 C CNN
 F 1 "+3V3" H 3000 6830 50  0000 C CNN
 F 2 "" H 3000 6700 50  0001 C CNN
@@
 $EndComp
 $Comp
-L GND #PWR053
+L GND #PWR050
 U 1 1 5933BE0C
 P 3000 7300
-F 0 "#PWR053" H 3000 7100 50  0001 C CNN
+F 0 "#PWR050" H 3000 7100 50  0001 C CNN
 F 1 "GND" H 3000 7175 30  0001 C CNN
 F 2 "" H 3000 7300 50  0001 C CNN
@@
 $EndComp
 $Comp
-L GND #PWR054
+L GND #PWR051
 U 1 1 5933BE19
 P 2650 7300
-F 0 "#PWR054" H 2650 7100 50  0001 C CNN
+F 0 "#PWR051" H 2650 7100 50  0001 C CNN
 F 1 "GND" H 2650 7175 30  0001 C CNN
 F 2 "" H 2650 7300 50  0001 C CNN
@@
 $EndComp
 $Comp
-L +3V3 #PWR055
+L +3V3 #PWR052
 U 1 1 5933BE1F
 P 2650 6700
-F 0 "#PWR055" H 2680 6730 10  0001 C CNN
+F 0 "#PWR052" H 2680 6730 10  0001 C CNN
 F 1 "+3V3" H 2650 6830 50  0000 C CNN
 F 2 "" H 2650 6700 50  0001 C CNN
@@
 $EndComp
 $Comp
-L +3V3 #PWR056
+L +3V3 #PWR053
 U 1 1 5943325E
 P 6100 5100
-F 0 "#PWR056" H 6130 5130 10  0001 C CNN
+F 0 "#PWR053" H 6130 5130 10  0001 C CNN
 F 1 "+3V3" H 6100 5230 50  0000 C CNN
 F 2 "" H 6100 5100 50  0001 C CNN
@@
 $EndComp
 $Comp
-L +3V3 #PWR057
+L +3V3 #PWR054
 U 1 1 59433264
 P 5700 5100
-F 0 "#PWR057" H 5730 5130 10  0001 C CNN
+F 0 "#PWR054" H 5730 5130 10  0001 C CNN
 F 1 "+3V3" H 5700 5230 50  0000 C CNN
 F 2 "" H 5700 5100 50  0001 C CNN
@@
 F 0 "RN3" V 5300 5450 60  0000 C CNN
 F 1 "R" V 5400 5450 40  0000 C CNN
-F 2 "pnRLC:4x0603_N" V 5550 5450 30  0001 C CNN
+F 2 "niceRLC:4x0603_N" V 5550 5450 30  0001 C CNN
 F 3 "" H 5400 5450 30  0000 C CNN
 	1    5400 5450
@@
 F 0 "RN3" V 5350 5300 40  0001 C CNN
 F 1 "R" V 5400 5550 40  0000 C CNN
-F 2 "pnRLC:4x0603_N" V 5550 5550 30  0001 C CNN
+F 2 "niceRLC:4x0603_N" V 5550 5550 30  0001 C CNN
 F 3 "" H 5400 5550 30  0000 C CNN
 	2    5400 5550
@@
 F 0 "RN3" V 5350 6350 40  0001 C CNN
 F 1 "R" V 5400 6600 40  0000 C CNN
-F 2 "pnRLC:4x0603_N" V 5550 6600 30  0001 C CNN
+F 2 "niceRLC:4x0603_N" V 5550 6600 30  0001 C CNN
 F 3 "" H 5400 6600 30  0000 C CNN
 	3    5400 6600
@@
 	4850 6600 5250 6600
 $Comp
-L +3V3 #PWR058
+L +3V3 #PWR055
 U 1 1 59433291
 P 6100 5950
-F 0 "#PWR058" H 6130 5980 10  0001 C CNN
+F 0 "#PWR055" H 6130 5980 10  0001 C CNN
 F 1 "+3V3" H 6100 6080 50  0000 C CNN
 F 2 "" H 6100 5950 50  0001 C CNN
@@
 $EndComp
 $Comp
-L +3V3 #PWR059
+L +3V3 #PWR056
 U 1 1 59433297
 P 5600 6000
-F 0 "#PWR059" H 5630 6030 10  0001 C CNN
+F 0 "#PWR056" H 5630 6030 10  0001 C CNN
 F 1 "+3V3" H 5600 6130 50  0000 C CNN
 F 2 "" H 5600 6000 50  0001 C CNN
@@
 F 0 "RN3" V 5300 6100 40  0001 C CNN
 F 1 "R" V 5350 6350 40  0000 C CNN
-F 2 "pnRLC:4x0603_N" V 5500 6350 30  0001 C CNN
+F 2 "niceRLC:4x0603_N" V 5500 6350 30  0001 C CNN
 F 3 "" H 5350 6350 30  0000 C CNN
 	4    5350 6350
 	0    1    1    0
 $EndComp
+$Comp
+L R_V R48
+U 1 1 59488419
+P 4900 3350
+F 0 "R48" H 4960 3390 60  0000 L CNN
+F 1 "10k" H 4960 3310 40  0000 L CNN
+F 2 "0603_R_N" H 4960 3250 40  0001 L CNN
+F 3 "" H 4900 3350 60  0001 C CNN
+	1    4900 3350
+	1    0    0    -1
+$EndComp
+$Comp
+L PDTA143ZT Q12
+U 1 1 59488420
+P 4800 2900
+F 0 "Q12" H 4925 2950 60  0000 L CNN
+F 1 "PDTA143ZT" H 4925 2850 40  0000 L CNN
+F 2 "niceSemiconductors:SOT23-3_N" H 4950 2800 20  0001 L CNN
+F 3 "" H 4795 2900 60  0000 C CNN
+	1    4800 2900
+	1    0    0    -1
+$EndComp
+Wire Wire Line
+	4900 3050 4900 3250
+$Comp
+L +3V3 #PWR057
+U 1 1 594889A8
+P 4900 2700
+F 0 "#PWR057" H 4930 2730 10  0001 C CNN
+F 1 "+3V3" H 4900 2830 50  0000 C CNN
+F 2 "" H 4900 2700 50  0001 C CNN
+F 3 "" H 4900 2700 50  0001 C CNN
+	1    4900 2700
+	1    0    0    -1
+$EndComp
+Wire Wire Line
+	4900 2700 4900 2750
+Connection ~ 4900 3150
+Wire Wire Line
+	5800 3050 5800 2550
+$Comp
+L GND #PWR058
+U 1 1 59488CCB
+P 4900 3500
+F 0 "#PWR058" H 4930 3470 10  0001 C CNN
+F 1 "GND" H 4900 3375 40  0001 C CNN
+F 2 "" H 4900 3500 50  0001 C CNN
+F 3 "" H 4900 3500 50  0001 C CNN
+	1    4900 3500
+	1    0    0    -1
+$EndComp
+Wire Wire Line
+	4900 3500 4900 3450
+Wire Wire Line
+	4650 2900 4400 2900
+Text HLabel 4400 2900 0    56   Input ~ 0
+~VDD1_EN
 $EndSCHEMATC
