File: kicad/front/SUPER_UART_front_RS232.sch (KiCad schematic (older format))
At the start: 28 parts, among them CON3 RS232, Q12 PDTA143ZT, SW18 DTR, SW19 RTS, U4 74HC08P, U5 MAX3243EIPW, U6 74HC08P

Commit message: Routing before moving to 4 layers
Connections:
- net CTS_D: now also U4.11 (OUT); no longer U6.6 (OUT)
- net CTS_D1: now also U4.13 (in2); no longer U6.4 (in1)
- net CTS_D2: now also U4.12 (in1); no longer U6.5 (in2)
- net DCD_D: now also U4.8 (OUT); no longer U4.11 (OUT)
- net DCD_D1: now also U4.9 (in1); no longer U4.12 (in1)
- net DCD_D2: now also U4.10 (in2); no longer U4.13 (in2)
- net DSR_D: now also U6.8 (OUT); no longer U4.8 (OUT)
- net DSR_D1: now also U6.9 (in1); no longer U4.9 (in1)
- net DSR_D2: now also U6.10 (in2); no longer U4.10 (in2)
- net DTR_D: now also U4.4 (in1); no longer U4.1 (in1)
- net DTR_D1: now also U4.6 (OUT); no longer U4.3 (OUT)
- net DTR_FORCE: now also U4.5 (in2); no longer U4.2 (in2)
- net RTS_D: now also U4.1 (in1); no longer U4.4 (in1)
- net RTS_D1: now also U4.3 (OUT); no longer U4.6 (OUT)
- net RTS_FORCE: now also U4.2 (in2); no longer U4.5 (in2)
- net RXD_D2: now also U6.4 (in1); no longer U6.9 (in1)
- net RXD_D3: now also U6.5 (in2); no longer U6.10 (in2)
- net at U6.2 (in2): now also U6.6 (OUT); no longer U6.8 (OUT)
Other:
- moved on the sheet: U4A, U4B, U4C, U4D, U6B, U6C
Changed lines of the file:
@@
 $EndComp
 $Comp
-L GND #PWR032
+L GND #PWR038
 U 1 1 5933AA2F
 P 5550 2900
-F 0 "#PWR032" H 5580 2870 10  0001 C CNN
+F 0 "#PWR038" H 5580 2870 10  0001 C CNN
 F 1 "GND" H 5550 2775 40  0001 C CNN
 F 2 "" H 5550 2900 50  0001 C CNN
@@
 $EndComp
 $Comp
-L +3V3 #PWR033
+L +3V3 #PWR039
 U 1 1 5933AA35
 P 5550 2500
-F 0 "#PWR033" H 5580 2530 10  0001 C CNN
+F 0 "#PWR039" H 5580 2530 10  0001 C CNN
 F 1 "+3V3" H 5550 2630 50  0000 C CNN
 F 2 "" H 5550 2500 50  0001 C CNN
@@
 $EndComp
 $Comp
-L GND #PWR034
+L GND #PWR040
 U 1 1 5933AA3B
 P 5550 3800
-F 0 "#PWR034" H 5580 3770 10  0001 C CNN
+F 0 "#PWR040" H 5580 3770 10  0001 C CNN
 F 1 "GND" H 5550 3675 40  0001 C CNN
 F 2 "" H 5550 3800 50  0001 C CNN
@@
 NoConn ~ 5900 3250
 $Comp
-L GND #PWR035
+L GND #PWR041
 U 1 1 5933AA42
 P 8050 3800
-F 0 "#PWR035" H 8080 3770 10  0001 C CNN
+F 0 "#PWR041" H 8080 3770 10  0001 C CNN
 F 1 "GND" H 8050 3675 40  0001 C CNN
 F 2 "" H 8050 3800 50  0001 C CNN
@@
 $EndComp
 $Comp
-L GND #PWR036
+L GND #PWR042
 U 1 1 5933AA67
 P 10600 3250
-F 0 "#PWR036" H 10630 3220 10  0001 C CNN
+F 0 "#PWR042" H 10630 3220 10  0001 C CNN
 F 1 "GND" H 10600 3125 40  0001 C CNN
 F 2 "" H 10600 3250 50  0001 C CNN
@@
 $EndComp
 $Comp
-L GND #PWR037
+L GND #PWR043
 U 1 1 5933AA74
 P 9950 3250
-F 0 "#PWR037" H 9980 3220 10  0001 C CNN
+F 0 "#PWR043" H 9980 3220 10  0001 C CNN
 F 1 "GND" H 9950 3125 40  0001 C CNN
 F 2 "" H 9950 3250 50  0001 C CNN
@@
 DTR_232
 $Comp
-L GND #PWR038
+L GND #PWR044
 U 1 1 5933AA89
 P 10300 2550
-F 0 "#PWR038" H 10330 2520 10  0001 C CNN
+F 0 "#PWR044" H 10330 2520 10  0001 C CNN
 F 1 "GND" H 10300 2425 40  0001 C CNN
 F 2 "" H 10300 2550 50  0001 C CNN
@@
 $EndComp
 $Comp
-L GND #PWR039
+L GND #PWR045
 U 1 1 5933BD74
 P 1650 2250
-F 0 "#PWR039" H 1650 2050 50  0001 C CNN
+F 0 "#PWR045" H 1650 2050 50  0001 C CNN
 F 1 "GND" H 1650 2125 30  0001 C CNN
 F 2 "" H 1650 2250 50  0001 C CNN
@@
 $EndComp
 $Comp
-L +3V3 #PWR040
+L +3V3 #PWR046
 U 1 1 5933BD81
 P 1650 1050
-F 0 "#PWR040" H 1680 1080 10  0001 C CNN
+F 0 "#PWR046" H 1680 1080 10  0001 C CNN
 F 1 "+3V3" H 1650 1180 50  0000 C CNN
 F 2 "" H 1650 1050 50  0001 C CNN
@@
 $EndComp
 $Comp
-L GND #PWR041
+L GND #PWR047
 U 1 1 5933BD88
 P 1650 3800
-F 0 "#PWR041" H 1650 3600 50  0001 C CNN
+F 0 "#PWR047" H 1650 3600 50  0001 C CNN
 F 1 "GND" H 1650 3675 30  0001 C CNN
 F 2 "" H 1650 3800 50  0001 C CNN
@@
 $EndComp
 $Comp
-L +3V3 #PWR042
+L +3V3 #PWR048
 U 1 1 5933BD95
 P 1650 2700
-F 0 "#PWR042" H 1680 2730 10  0001 C CNN
+F 0 "#PWR048" H 1680 2730 10  0001 C CNN
 F 1 "+3V3" H 1650 2830 50  0000 C CNN
 F 2 "" H 1650 2700 50  0001 C CNN
@@
 $EndComp
 $Comp
-L +3V3 #PWR043
+L +3V3 #PWR049
 U 1 1 5933BDC9
 P 2250 2700
-F 0 "#PWR043" H 2280 2730 10  0001 C CNN
+F 0 "#PWR049" H 2280 2730 10  0001 C CNN
 F 1 "+3V3" H 2250 2830 50  0000 C CNN
 F 2 "" H 2250 2700 50  0001 C CNN
@@
 $EndComp
 $Comp
-L +3V3 #PWR044
+L +3V3 #PWR050
 U 1 1 5933BDD9
 P 2250 1050
-F 0 "#PWR044" H 2280 1080 10  0001 C CNN
+F 0 "#PWR050" H 2280 1080 10  0001 C CNN
 F 1 "+3V3" H 2250 1180 50  0000 C CNN
 F 2 "" H 2250 1050 50  0001 C CNN
@@
 	1650 1800 2450 1800
 $Comp
-L +3V3 #PWR045
+L +3V3 #PWR051
 U 1 1 5933BDE3
 P 2100 6700
-F 0 "#PWR045" H 2130 6730 10  0001 C CNN
+F 0 "#PWR051" H 2130 6730 10  0001 C CNN
 F 1 "+3V3" H 2100 6830 50  0000 C CNN
 F 2 "" H 2100 6700 50  0001 C CNN
@@
 $EndComp
 $Comp
-L GND #PWR046
+L GND #PWR052
 U 1 1 5933BDE9
 P 2100 7300
-F 0 "#PWR046" H 2100 7100 50  0001 C CNN
+F 0 "#PWR052" H 2100 7100 50  0001 C CNN
 F 1 "GND" H 2100 7175 30  0001 C CNN
 F 2 "" H 2100 7300 50  0001 C CNN
@@
 $EndComp
 $Comp
-L GND #PWR047
+L GND #PWR053
 U 1 1 5933BDF6
 P 1750 7300
-F 0 "#PWR047" H 1750 7100 50  0001 C CNN
+F 0 "#PWR053" H 1750 7100 50  0001 C CNN
 F 1 "GND" H 1750 7175 30  0001 C CNN
 F 2 "" H 1750 7300 50  0001 C CNN
@@
 $EndComp
 $Comp
-L +3V3 #PWR048
+L +3V3 #PWR054
 U 1 1 5933BDFC
 P 1750 6700
-F 0 "#PWR048" H 1780 6730 10  0001 C CNN
+F 0 "#PWR054" H 1780 6730 10  0001 C CNN
 F 1 "+3V3" H 1750 6830 50  0000 C CNN
 F 2 "" H 1750 6700 50  0001 C CNN
@@
 	2100 6750 2100 6700
 $Comp
-L +3V3 #PWR049
+L +3V3 #PWR055
 U 1 1 5933BE06
 P 3000 6700
-F 0 "#PWR049" H 3030 6730 10  0001 C CNN
+F 0 "#PWR055" H 3030 6730 10  0001 C CNN
 F 1 "+3V3" H 3000 6830 50  0000 C CNN
 F 2 "" H 3000 6700 50  0001 C CNN
@@
 $EndComp
 $Comp
-L GND #PWR050
+L GND #PWR056
 U 1 1 5933BE0C
 P 3000 7300
-F 0 "#PWR050" H 3000 7100 50  0001 C CNN
+F 0 "#PWR056" H 3000 7100 50  0001 C CNN
 F 1 "GND" H 3000 7175 30  0001 C CNN
 F 2 "" H 3000 7300 50  0001 C CNN
@@
 $EndComp
 $Comp
-L GND #PWR051
+L GND #PWR057
 U 1 1 5933BE19
 P 2650 7300
-F 0 "#PWR051" H 2650 7100 50  0001 C CNN
+F 0 "#PWR057" H 2650 7100 50  0001 C CNN
 F 1 "GND" H 2650 7175 30  0001 C CNN
 F 2 "" H 2650 7300 50  0001 C CNN
@@
 $EndComp
 $Comp
-L +3V3 #PWR052
+L +3V3 #PWR058
 U 1 1 5933BE1F
 P 2650 6700
-F 0 "#PWR052" H 2680 6730 10  0001 C CNN
+F 0 "#PWR058" H 2680 6730 10  0001 C CNN
 F 1 "+3V3" H 2650 6830 50  0000 C CNN
 F 2 "" H 2650 6700 50  0001 C CNN
@@
 L 74HC08P U4
 U 3 1 5933BE31
-P 2200 4450
-F 0 "U4" H 2200 4600 60  0000 C CNN
-F 1 "74HC08P" H 2200 4300 40  0000 C CNN
-F 2 "niceSemiconductors:TSSOP-14_N" H 2300 4290 40  0001 L CNN
-F 3 "" H 2200 4450 60  0001 C CNN
-	3    2200 4450
+P 2200 4850
+F 0 "U4" H 2200 5000 60  0000 C CNN
+F 1 "74HC08P" H 2200 4700 40  0000 C CNN
+F 2 "niceSemiconductors:TSSOP-14_N" H 2300 4690 40  0001 L CNN
+F 3 "" H 2200 4850 60  0001 C CNN
+	3    2200 4850
 	-1   0    0    -1
 $EndComp
@@
 L 74HC08P U6
 U 2 1 5933BE3F
-P 2200 5850
-F 0 "U6" H 2200 6000 60  0000 C CNN
-F 1 "74HC08P" H 2200 5700 40  0000 C CNN
-F 2 "niceSemiconductors:TSSOP-14_N" H 2300 5690 40  0001 L CNN
-F 3 "" H 2200 5850 60  0001 C CNN
-	2    2200 5850
+P 2750 5450
+F 0 "U6" H 2750 5600 60  0000 C CNN
+F 1 "74HC08P" H 2750 5300 40  0000 C CNN
+F 2 "niceSemiconductors:TSSOP-14_N" H 2850 5290 40  0001 L CNN
+F 3 "" H 2750 5450 60  0001 C CNN
+	2    2750 5450
 	-1   0    0    -1
 $EndComp
@@
 L 74HC08P U4
 U 1 1 5933BE46
-P 2650 1750
-F 0 "U4" H 2650 1900 60  0000 C CNN
-F 1 "74HC08P" H 2650 1600 40  0000 C CNN
-F 2 "niceSemiconductors:TSSOP-14_N" H 2750 1590 40  0001 L CNN
-F 3 "" H 2650 1750 60  0001 C CNN
-	1    2650 1750
+P 2650 3300
+F 0 "U4" H 2650 3450 60  0000 C CNN
+F 1 "74HC08P" H 2650 3150 40  0000 C CNN
+F 2 "niceSemiconductors:TSSOP-14_N" H 2750 3140 40  0001 L CNN
+F 3 "" H 2650 3300 60  0001 C CNN
+	1    2650 3300
 	1    0    0    -1
 $EndComp
@@
 L 74HC08P U4
 U 4 1 5933BE54
-P 2200 4850
-F 0 "U4" H 2200 5000 60  0000 C CNN
-F 1 "74HC08P" H 2200 4700 40  0000 C CNN
-F 2 "niceSemiconductors:TSSOP-14_N" H 2300 4690 40  0001 L CNN
-F 3 "" H 2200 4850 60  0001 C CNN
-	4    2200 4850
-	-1   0    0    -1
+P 2200 5850
+F 0 "U4" H 2200 6000 60  0000 C CNN
+F 1 "74HC08P" H 2200 5700 40  0000 C CNN
+F 2 "niceSemiconductors:TSSOP-14_N" H 2300 5690 40  0001 L CNN
+F 3 "" H 2200 5850 60  0001 C CNN
+	4    2200 5850
+	-1   0    0    1
 $EndComp
 $Comp
@@
 L 74HC08P U4
 U 2 1 5933BE69
-P 2650 3300
-F 0 "U4" H 2650 3450 60  0000 C CNN
-F 1 "74HC08P" H 2650 3150 40  0000 C CNN
-F 2 "niceSemiconductors:TSSOP-14_N" H 2750 3140 40  0001 L CNN
-F 3 "" H 2650 3300 60  0001 C CNN
-	2    2650 3300
+P 2650 1750
+F 0 "U4" H 2650 1900 60  0000 C CNN
+F 1 "74HC08P" H 2650 1600 40  0000 C CNN
+F 2 "niceSemiconductors:TSSOP-14_N" H 2750 1590 40  0001 L CNN
+F 3 "" H 2650 1750 60  0001 C CNN
+	2    2650 1750
 	1    0    0    -1
 $EndComp
@@
 L 74HC08P U6
 U 3 1 5934E9A6
-P 2750 5450
-F 0 "U6" H 2750 5600 60  0000 C CNN
-F 1 "74HC08P" H 2750 5300 40  0000 C CNN
-F 2 "niceSemiconductors:TSSOP-14_N" H 2850 5290 40  0001 L CNN
-F 3 "" H 2750 5450 60  0001 C CNN
-	3    2750 5450
+P 2200 4450
+F 0 "U6" H 2200 4600 60  0000 C CNN
+F 1 "74HC08P" H 2200 4300 40  0000 C CNN
+F 2 "niceSemiconductors:TSSOP-14_N" H 2300 4290 40  0001 L CNN
+F 3 "" H 2200 4450 60  0001 C CNN
+	3    2200 4450
 	-1   0    0    -1
 $EndComp
@@
 $EndComp
 $Comp
-L +3V3 #PWR053
+L +3V3 #PWR059
 U 1 1 5943325E
 P 6100 5100
-F 0 "#PWR053" H 6130 5130 10  0001 C CNN
+F 0 "#PWR059" H 6130 5130 10  0001 C CNN
 F 1 "+3V3" H 6100 5230 50  0000 C CNN
 F 2 "" H 6100 5100 50  0001 C CNN
@@
 $EndComp
 $Comp
-L +3V3 #PWR054
+L +3V3 #PWR060
 U 1 1 59433264
 P 5700 5100
-F 0 "#PWR054" H 5730 5130 10  0001 C CNN
+F 0 "#PWR060" H 5730 5130 10  0001 C CNN
 F 1 "+3V3" H 5700 5230 50  0000 C CNN
 F 2 "" H 5700 5100 50  0001 C CNN
@@
 	4850 6600 5250 6600
 $Comp
-L +3V3 #PWR055
+L +3V3 #PWR061
 U 1 1 59433291
 P 6100 5950
-F 0 "#PWR055" H 6130 5980 10  0001 C CNN
+F 0 "#PWR061" H 6130 5980 10  0001 C CNN
 F 1 "+3V3" H 6100 6080 50  0000 C CNN
 F 2 "" H 6100 5950 50  0001 C CNN
@@
 $EndComp
 $Comp
-L +3V3 #PWR056
+L +3V3 #PWR062
 U 1 1 59433297
 P 5600 6000
-F 0 "#PWR056" H 5630 6030 10  0001 C CNN
+F 0 "#PWR062" H 5630 6030 10  0001 C CNN
 F 1 "+3V3" H 5600 6130 50  0000 C CNN
 F 2 "" H 5600 6000 50  0001 C CNN
@@
 	4900 3050 4900 3250
 $Comp
-L +3V3 #PWR057
+L +3V3 #PWR063
 U 1 1 594889A8
 P 4900 2700
-F 0 "#PWR057" H 4930 2730 10  0001 C CNN
+F 0 "#PWR063" H 4930 2730 10  0001 C CNN
 F 1 "+3V3" H 4900 2830 50  0000 C CNN
 F 2 "" H 4900 2700 50  0001 C CNN
@@
 	5800 3050 5800 2550
 $Comp
-L GND #PWR058
+L GND #PWR064
 U 1 1 59488CCB
 P 4900 3500
-F 0 "#PWR058" H 4930 3470 10  0001 C CNN
+F 0 "#PWR064" H 4930 3470 10  0001 C CNN
 F 1 "GND" H 4900 3375 40  0001 C CNN
 F 2 "" H 4900 3500 50  0001 C CNN

Commit message: Front board routed
Parts:
- removed C18: 100n, 0603_N, symbol C
Changed lines of the file:
@@
 $EndComp
 $Comp
-L GND #PWR038
+L GND #PWR040
 U 1 1 5933AA2F
 P 5550 2900
-F 0 "#PWR038" H 5580 2870 10  0001 C CNN
+F 0 "#PWR040" H 5580 2870 10  0001 C CNN
 F 1 "GND" H 5550 2775 40  0001 C CNN
 F 2 "" H 5550 2900 50  0001 C CNN
@@
 $EndComp
 $Comp
-L +3V3 #PWR039
+L +3V3 #PWR041
 U 1 1 5933AA35
 P 5550 2500
-F 0 "#PWR039" H 5580 2530 10  0001 C CNN
+F 0 "#PWR041" H 5580 2530 10  0001 C CNN
 F 1 "+3V3" H 5550 2630 50  0000 C CNN
 F 2 "" H 5550 2500 50  0001 C CNN
@@
 $EndComp
 $Comp
-L GND #PWR040
+L GND #PWR042
 U 1 1 5933AA3B
 P 5550 3800
-F 0 "#PWR040" H 5580 3770 10  0001 C CNN
+F 0 "#PWR042" H 5580 3770 10  0001 C CNN
 F 1 "GND" H 5550 3675 40  0001 C CNN
 F 2 "" H 5550 3800 50  0001 C CNN
@@
 NoConn ~ 5900 3250
 $Comp
-L GND #PWR041
+L GND #PWR043
 U 1 1 5933AA42
 P 8050 3800
-F 0 "#PWR041" H 8080 3770 10  0001 C CNN
+F 0 "#PWR043" H 8080 3770 10  0001 C CNN
 F 1 "GND" H 8050 3675 40  0001 C CNN
 F 2 "" H 8050 3800 50  0001 C CNN
@@
 $EndComp
 $Comp
-L GND #PWR042
+L GND #PWR044
 U 1 1 5933AA67
 P 10600 3250
-F 0 "#PWR042" H 10630 3220 10  0001 C CNN
+F 0 "#PWR044" H 10630 3220 10  0001 C CNN
 F 1 "GND" H 10600 3125 40  0001 C CNN
 F 2 "" H 10600 3250 50  0001 C CNN
@@
 $EndComp
 $Comp
-L GND #PWR043
+L GND #PWR045
 U 1 1 5933AA74
 P 9950 3250
-F 0 "#PWR043" H 9980 3220 10  0001 C CNN
+F 0 "#PWR045" H 9980 3220 10  0001 C CNN
 F 1 "GND" H 9950 3125 40  0001 C CNN
 F 2 "" H 9950 3250 50  0001 C CNN
@@
 DTR_232
 $Comp
-L GND #PWR044
+L GND #PWR046
 U 1 1 5933AA89
 P 10300 2550
-F 0 "#PWR044" H 10330 2520 10  0001 C CNN
+F 0 "#PWR046" H 10330 2520 10  0001 C CNN
 F 1 "GND" H 10300 2425 40  0001 C CNN
 F 2 "" H 10300 2550 50  0001 C CNN
@@
 $EndComp
 $Comp
-L GND #PWR045
+L GND #PWR047
 U 1 1 5933BD74
 P 1650 2250
-F 0 "#PWR045" H 1650 2050 50  0001 C CNN
+F 0 "#PWR047" H 1650 2050 50  0001 C CNN
 F 1 "GND" H 1650 2125 30  0001 C CNN
 F 2 "" H 1650 2250 50  0001 C CNN
@@
 $EndComp
 $Comp
-L +3V3 #PWR046
+L +3V3 #PWR048
 U 1 1 5933BD81
 P 1650 1050
-F 0 "#PWR046" H 1680 1080 10  0001 C CNN
+F 0 "#PWR048" H 1680 1080 10  0001 C CNN
 F 1 "+3V3" H 1650 1180 50  0000 C CNN
 F 2 "" H 1650 1050 50  0001 C CNN
@@
 $EndComp
 $Comp
-L GND #PWR047
+L GND #PWR049
 U 1 1 5933BD88
 P 1650 3800
-F 0 "#PWR047" H 1650 3600 50  0001 C CNN
+F 0 "#PWR049" H 1650 3600 50  0001 C CNN
 F 1 "GND" H 1650 3675 30  0001 C CNN
 F 2 "" H 1650 3800 50  0001 C CNN
@@
 $EndComp
 $Comp
-L +3V3 #PWR048
+L +3V3 #PWR050
 U 1 1 5933BD95
 P 1650 2700
-F 0 "#PWR048" H 1680 2730 10  0001 C CNN
+F 0 "#PWR050" H 1680 2730 10  0001 C CNN
 F 1 "+3V3" H 1650 2830 50  0000 C CNN
 F 2 "" H 1650 2700 50  0001 C CNN
@@
 $EndComp
 $Comp
-L +3V3 #PWR049
+L +3V3 #PWR051
 U 1 1 5933BDC9
 P 2250 2700
-F 0 "#PWR049" H 2280 2730 10  0001 C CNN
+F 0 "#PWR051" H 2280 2730 10  0001 C CNN
 F 1 "+3V3" H 2250 2830 50  0000 C CNN
 F 2 "" H 2250 2700 50  0001 C CNN
@@
 $EndComp
 $Comp
-L +3V3 #PWR050
+L +3V3 #PWR052
 U 1 1 5933BDD9
 P 2250 1050
-F 0 "#PWR050" H 2280 1080 10  0001 C CNN
+F 0 "#PWR052" H 2280 1080 10  0001 C CNN
 F 1 "+3V3" H 2250 1180 50  0000 C CNN
 F 2 "" H 2250 1050 50  0001 C CNN
@@
 	1650 1800 2450 1800
 $Comp
-L +3V3 #PWR051
+L +3V3 #PWR053
 U 1 1 5933BDE3
 P 2100 6700
-F 0 "#PWR051" H 2130 6730 10  0001 C CNN
+F 0 "#PWR053" H 2130 6730 10  0001 C CNN
 F 1 "+3V3" H 2100 6830 50  0000 C CNN
 F 2 "" H 2100 6700 50  0001 C CNN
@@
 $EndComp
 $Comp
-L GND #PWR052
+L GND #PWR054
 U 1 1 5933BDE9
 P 2100 7300
-F 0 "#PWR052" H 2100 7100 50  0001 C CNN
+F 0 "#PWR054" H 2100 7100 50  0001 C CNN
 F 1 "GND" H 2100 7175 30  0001 C CNN
 F 2 "" H 2100 7300 50  0001 C CNN
@@
 $EndComp
 $Comp
-L GND #PWR053
+L GND #PWR055
 U 1 1 5933BDF6
 P 1750 7300
-F 0 "#PWR053" H 1750 7100 50  0001 C CNN
+F 0 "#PWR055" H 1750 7100 50  0001 C CNN
 F 1 "GND" H 1750 7175 30  0001 C CNN
 F 2 "" H 1750 7300 50  0001 C CNN
@@
 $EndComp
 $Comp
-L +3V3 #PWR054
+L +3V3 #PWR056
 U 1 1 5933BDFC
 P 1750 6700
-F 0 "#PWR054" H 1780 6730 10  0001 C CNN
+F 0 "#PWR056" H 1780 6730 10  0001 C CNN
 F 1 "+3V3" H 1750 6830 50  0000 C CNN
 F 2 "" H 1750 6700 50  0001 C CNN
@@
 	2100 6750 2100 6700
 $Comp
-L +3V3 #PWR055
+L +3V3 #PWR057
 U 1 1 5933BE06
 P 3000 6700
-F 0 "#PWR055" H 3030 6730 10  0001 C CNN
+F 0 "#PWR057" H 3030 6730 10  0001 C CNN
 F 1 "+3V3" H 3000 6830 50  0000 C CNN
 F 2 "" H 3000 6700 50  0001 C CNN
@@
 $EndComp
 $Comp
-L GND #PWR056
+L GND #PWR058
 U 1 1 5933BE0C
 P 3000 7300
-F 0 "#PWR056" H 3000 7100 50  0001 C CNN
+F 0 "#PWR058" H 3000 7100 50  0001 C CNN
 F 1 "GND" H 3000 7175 30  0001 C CNN
 F 2 "" H 3000 7300 50  0001 C CNN
@@
 $EndComp
 $Comp
-L C C18
-U 1 1 5933BE12
-P 2650 7000
-F 0 "C18" H 2670 7100 60  0000 L CNN
-F 1 "100n" H 2670 6900 40  0000 L CNN
-F 2 "0603_N" H 2670 6840 40  0001 L CNN
-F 3 "" H 2650 7000 60  0001 C CNN
-	1    2650 7000
-	1    0    0    -1
-$EndComp
-$Comp
-L GND #PWR057
+L GND #PWR059
 U 1 1 5933BE19
 P 2650 7300
-F 0 "#PWR057" H 2650 7100 50  0001 C CNN
+F 0 "#PWR059" H 2650 7100 50  0001 C CNN
 F 1 "GND" H 2650 7175 30  0001 C CNN
 F 2 "" H 2650 7300 50  0001 C CNN
@@
 $EndComp
 $Comp
-L +3V3 #PWR058
+L +3V3 #PWR060
 U 1 1 5933BE1F
 P 2650 6700
-F 0 "#PWR058" H 2680 6730 10  0001 C CNN
+F 0 "#PWR060" H 2680 6730 10  0001 C CNN
 F 1 "+3V3" H 2650 6830 50  0000 C CNN
 F 2 "" H 2650 6700 50  0001 C CNN
@@
 $EndComp
 $Comp
-L +3V3 #PWR059
+L +3V3 #PWR061
 U 1 1 5943325E
 P 6100 5100
-F 0 "#PWR059" H 6130 5130 10  0001 C CNN
+F 0 "#PWR061" H 6130 5130 10  0001 C CNN
 F 1 "+3V3" H 6100 5230 50  0000 C CNN
 F 2 "" H 6100 5100 50  0001 C CNN
@@
 $EndComp
 $Comp
-L +3V3 #PWR060
+L +3V3 #PWR062
 U 1 1 59433264
 P 5700 5100
-F 0 "#PWR060" H 5730 5130 10  0001 C CNN
+F 0 "#PWR062" H 5730 5130 10  0001 C CNN
 F 1 "+3V3" H 5700 5230 50  0000 C CNN
 F 2 "" H 5700 5100 50  0001 C CNN
@@
 	4850 6600 5250 6600
 $Comp
-L +3V3 #PWR061
+L +3V3 #PWR063
 U 1 1 59433291
 P 6100 5950
-F 0 "#PWR061" H 6130 5980 10  0001 C CNN
+F 0 "#PWR063" H 6130 5980 10  0001 C CNN
 F 1 "+3V3" H 6100 6080 50  0000 C CNN
 F 2 "" H 6100 5950 50  0001 C CNN
@@
 $EndComp
 $Comp
-L +3V3 #PWR062
+L +3V3 #PWR064
 U 1 1 59433297
 P 5600 6000
-F 0 "#PWR062" H 5630 6030 10  0001 C CNN
+F 0 "#PWR064" H 5630 6030 10  0001 C CNN
 F 1 "+3V3" H 5600 6130 50  0000 C CNN
 F 2 "" H 5600 6000 50  0001 C CNN
@@
 	4900 3050 4900 3250
 $Comp
-L +3V3 #PWR063
+L +3V3 #PWR065
 U 1 1 594889A8
 P 4900 2700
-F 0 "#PWR063" H 4930 2730 10  0001 C CNN
+F 0 "#PWR065" H 4930 2730 10  0001 C CNN
 F 1 "+3V3" H 4900 2830 50  0000 C CNN
 F 2 "" H 4900 2700 50  0001 C CNN
@@
 	5800 3050 5800 2550
 $Comp
-L GND #PWR064
+L GND #PWR066
 U 1 1 59488CCB
 P 4900 3500
-F 0 "#PWR064" H 4930 3470 10  0001 C CNN
+F 0 "#PWR066" H 4930 3470 10  0001 C CNN
 F 1 "GND" H 4900 3375 40  0001 C CNN
 F 2 "" H 4900 3500 50  0001 C CNN
