File: kicad/front/SUPER_UART_front_RS232.sch (KiCad schematic (older format))
At the start: 27 parts, among them CON3 RS232, Q12 PDTA143ZT, SW18 DTR, SW19 RTS, U4 74HC08P, U5 MAX3243EIPW, U6 74HC08P

Commit message: Add missing files
Parts:
- R3, R5: value R -> 220R
- RN3: value R -> 1k
Other:
- note added: "Add some ESD caps"
Changed lines of the file:
@@
 EESchema Schematic File Version 2
+LIBS:SUPER_UART_front-rescue
 LIBS:_test_
 LIBS:niceAVR
@@
 encoding utf-8
 Sheet 3 5
-Title ""
-Date ""
-Rev ""
-Comp ""
+Title "USB-UART converter"
+Date "2017-07-16"
+Rev "1"
+Comp "nicecircuits.com"
 Comment1 ""
 Comment2 ""
@@
 $EndComp
 $Comp
-L GND #PWR040
+L GND #PWR046
 U 1 1 5933AA2F
 P 5550 2900
-F 0 "#PWR040" H 5580 2870 10  0001 C CNN
+F 0 "#PWR046" H 5580 2870 10  0001 C CNN
 F 1 "GND" H 5550 2775 40  0001 C CNN
 F 2 "" H 5550 2900 50  0001 C CNN
@@
 $EndComp
 $Comp
-L +3V3 #PWR041
+L +3V3-RESCUE-SUPER_UART_front #PWR047
 U 1 1 5933AA35
 P 5550 2500
-F 0 "#PWR041" H 5580 2530 10  0001 C CNN
+AR Path="/5933AA35" Ref="#PWR047"  Part="1"
+AR Path="/5933A622/5933AA35" Ref="#PWR047"  Part="1"
+F 0 "#PWR047" H 5580 2530 10  0001 C CNN
 F 1 "+3V3" H 5550 2630 50  0000 C CNN
 F 2 "" H 5550 2500 50  0001 C CNN
@@
 $EndComp
 $Comp
-L GND #PWR042
+L GND #PWR048
 U 1 1 5933AA3B
 P 5550 3800
-F 0 "#PWR042" H 5580 3770 10  0001 C CNN
+F 0 "#PWR048" H 5580 3770 10  0001 C CNN
 F 1 "GND" H 5550 3675 40  0001 C CNN
 F 2 "" H 5550 3800 50  0001 C CNN
@@
 NoConn ~ 5900 3250
 $Comp
-L GND #PWR043
+L GND #PWR049
 U 1 1 5933AA42
 P 8050 3800
-F 0 "#PWR043" H 8080 3770 10  0001 C CNN
+F 0 "#PWR049" H 8080 3770 10  0001 C CNN
 F 1 "GND" H 8050 3675 40  0001 C CNN
 F 2 "" H 8050 3800 50  0001 C CNN
@@
 $EndComp
 $Comp
-L GND #PWR044
+L GND #PWR050
 U 1 1 5933AA67
 P 10600 3250
-F 0 "#PWR044" H 10630 3220 10  0001 C CNN
+F 0 "#PWR050" H 10630 3220 10  0001 C CNN
 F 1 "GND" H 10600 3125 40  0001 C CNN
 F 2 "" H 10600 3250 50  0001 C CNN
@@
 $EndComp
 $Comp
-L GND #PWR045
+L GND #PWR051
 U 1 1 5933AA74
 P 9950 3250
-F 0 "#PWR045" H 9980 3220 10  0001 C CNN
+F 0 "#PWR051" H 9980 3220 10  0001 C CNN
 F 1 "GND" H 9950 3125 40  0001 C CNN
 F 2 "" H 9950 3250 50  0001 C CNN
@@
 DTR_232
 $Comp
-L GND #PWR046
+L GND #PWR052
 U 1 1 5933AA89
 P 10300 2550
-F 0 "#PWR046" H 10330 2520 10  0001 C CNN
+F 0 "#PWR052" H 10330 2520 10  0001 C CNN
 F 1 "GND" H 10300 2425 40  0001 C CNN
 F 2 "" H 10300 2550 50  0001 C CNN
@@
 $EndComp
 $Comp
-L GND #PWR047
+L GND #PWR053
 U 1 1 5933BD74
 P 1650 2250
-F 0 "#PWR047" H 1650 2050 50  0001 C CNN
+F 0 "#PWR053" H 1650 2050 50  0001 C CNN
 F 1 "GND" H 1650 2125 30  0001 C CNN
 F 2 "" H 1650 2250 50  0001 C CNN
@@
 P 1650 1200
 F 0 "R3" H 1710 1240 60  0000 L CNN
-F 1 "R" H 1710 1160 40  0000 L CNN
+F 1 "220R" H 1710 1160 40  0000 L CNN
 F 2 "0603_R_N" H 1710 1100 40  0001 L CNN
 F 3 "" H 1650 1200 60  0001 C CNN
@@
 $EndComp
 $Comp
-L +3V3 #PWR048
+L +3V3-RESCUE-SUPER_UART_front #PWR054
 U 1 1 5933BD81
 P 1650 1050
-F 0 "#PWR048" H 1680 1080 10  0001 C CNN
+AR Path="/5933BD81" Ref="#PWR054"  Part="1"
+AR Path="/5933A622/5933BD81" Ref="#PWR054"  Part="1"
+F 0 "#PWR054" H 1680 1080 10  0001 C CNN
 F 1 "+3V3" H 1650 1180 50  0000 C CNN
 F 2 "" H 1650 1050 50  0001 C CNN
@@
 $EndComp
 $Comp
-L GND #PWR049
+L GND #PWR055
 U 1 1 5933BD88
 P 1650 3800
-F 0 "#PWR049" H 1650 3600 50  0001 C CNN
+F 0 "#PWR055" H 1650 3600 50  0001 C CNN
 F 1 "GND" H 1650 3675 30  0001 C CNN
 F 2 "" H 1650 3800 50  0001 C CNN
@@
 P 1650 2850
 F 0 "R5" H 1710 2890 60  0000 L CNN
-F 1 "R" H 1710 2810 40  0000 L CNN
+F 1 "220R" H 1710 2810 40  0000 L CNN
 F 2 "0603_R_N" H 1710 2750 40  0001 L CNN
 F 3 "" H 1650 2850 60  0001 C CNN
@@
 $EndComp
 $Comp
-L +3V3 #PWR050
+L +3V3-RESCUE-SUPER_UART_front #PWR056
 U 1 1 5933BD95
 P 1650 2700
-F 0 "#PWR050" H 1680 2730 10  0001 C CNN
+AR Path="/5933BD95" Ref="#PWR056"  Part="1"
+AR Path="/5933A622/5933BD95" Ref="#PWR056"  Part="1"
+F 0 "#PWR056" H 1680 2730 10  0001 C CNN
 F 1 "+3V3" H 1650 2830 50  0000 C CNN
 F 2 "" H 1650 2700 50  0001 C CNN
@@
 $EndComp
 $Comp
-L +3V3 #PWR051
+L +3V3-RESCUE-SUPER_UART_front #PWR057
 U 1 1 5933BDC9
 P 2250 2700
-F 0 "#PWR051" H 2280 2730 10  0001 C CNN
+AR Path="/5933BDC9" Ref="#PWR057"  Part="1"
+AR Path="/5933A622/5933BDC9" Ref="#PWR057"  Part="1"
+F 0 "#PWR057" H 2280 2730 10  0001 C CNN
 F 1 "+3V3" H 2250 2830 50  0000 C CNN
 F 2 "" H 2250 2700 50  0001 C CNN
@@
 $EndComp
 $Comp
-L +3V3 #PWR052
+L +3V3-RESCUE-SUPER_UART_front #PWR058
 U 1 1 5933BDD9
 P 2250 1050
-F 0 "#PWR052" H 2280 1080 10  0001 C CNN
+AR Path="/5933BDD9" Ref="#PWR058"  Part="1"
+AR Path="/5933A622/5933BDD9" Ref="#PWR058"  Part="1"
+F 0 "#PWR058" H 2280 1080 10  0001 C CNN
 F 1 "+3V3" H 2250 1180 50  0000 C CNN
 F 2 "" H 2250 1050 50  0001 C CNN
@@
 	1650 1800 2450 1800
 $Comp
-L +3V3 #PWR053
+L +3V3-RESCUE-SUPER_UART_front #PWR059
 U 1 1 5933BDE3
 P 2100 6700
-F 0 "#PWR053" H 2130 6730 10  0001 C CNN
+AR Path="/5933BDE3" Ref="#PWR059"  Part="1"
+AR Path="/5933A622/5933BDE3" Ref="#PWR059"  Part="1"
+F 0 "#PWR059" H 2130 6730 10  0001 C CNN
 F 1 "+3V3" H 2100 6830 50  0000 C CNN
 F 2 "" H 2100 6700 50  0001 C CNN
@@
 $EndComp
 $Comp
-L GND #PWR054
+L GND #PWR060
 U 1 1 5933BDE9
 P 2100 7300
-F 0 "#PWR054" H 2100 7100 50  0001 C CNN
+F 0 "#PWR060" H 2100 7100 50  0001 C CNN
 F 1 "GND" H 2100 7175 30  0001 C CNN
 F 2 "" H 2100 7300 50  0001 C CNN
@@
 $EndComp
 $Comp
-L GND #PWR055
+L GND #PWR061
 U 1 1 5933BDF6
 P 1750 7300
-F 0 "#PWR055" H 1750 7100 50  0001 C CNN
+F 0 "#PWR061" H 1750 7100 50  0001 C CNN
 F 1 "GND" H 1750 7175 30  0001 C CNN
 F 2 "" H 1750 7300 50  0001 C CNN
@@
 $EndComp
 $Comp
-L +3V3 #PWR056
+L +3V3-RESCUE-SUPER_UART_front #PWR062
 U 1 1 5933BDFC
 P 1750 6700
-F 0 "#PWR056" H 1780 6730 10  0001 C CNN
+AR Path="/5933BDFC" Ref="#PWR062"  Part="1"
+AR Path="/5933A622/5933BDFC" Ref="#PWR062"  Part="1"
+F 0 "#PWR062" H 1780 6730 10  0001 C CNN
 F 1 "+3V3" H 1750 6830 50  0000 C CNN
 F 2 "" H 1750 6700 50  0001 C CNN
@@
 	2100 6750 2100 6700
 $Comp
-L +3V3 #PWR057
+L +3V3-RESCUE-SUPER_UART_front #PWR063
 U 1 1 5933BE06
 P 3000 6700
-F 0 "#PWR057" H 3030 6730 10  0001 C CNN
+AR Path="/5933BE06" Ref="#PWR063"  Part="1"
+AR Path="/5933A622/5933BE06" Ref="#PWR063"  Part="1"
+F 0 "#PWR063" H 3030 6730 10  0001 C CNN
 F 1 "+3V3" H 3000 6830 50  0000 C CNN
 F 2 "" H 3000 6700 50  0001 C CNN
@@
 $EndComp
 $Comp
-L GND #PWR058
+L GND #PWR064
 U 1 1 5933BE0C
 P 3000 7300
-F 0 "#PWR058" H 3000 7100 50  0001 C CNN
+F 0 "#PWR064" H 3000 7100 50  0001 C CNN
 F 1 "GND" H 3000 7175 30  0001 C CNN
 F 2 "" H 3000 7300 50  0001 C CNN
@@
 $EndComp
 $Comp
-L GND #PWR059
+L GND #PWR065
 U 1 1 5933BE19
 P 2650 7300
-F 0 "#PWR059" H 2650 7100 50  0001 C CNN
+F 0 "#PWR065" H 2650 7100 50  0001 C CNN
 F 1 "GND" H 2650 7175 30  0001 C CNN
 F 2 "" H 2650 7300 50  0001 C CNN
@@
 $EndComp
 $Comp
-L +3V3 #PWR060
+L +3V3-RESCUE-SUPER_UART_front #PWR066
 U 1 1 5933BE1F
 P 2650 6700
-F 0 "#PWR060" H 2680 6730 10  0001 C CNN
+AR Path="/5933BE1F" Ref="#PWR066"  Part="1"
+AR Path="/5933A622/5933BE1F" Ref="#PWR066"  Part="1"
+F 0 "#PWR066" H 2680 6730 10  0001 C CNN
 F 1 "+3V3" H 2650 6830 50  0000 C CNN
 F 2 "" H 2650 6700 50  0001 C CNN
@@
 $EndComp
 $Comp
-L +3V3 #PWR061
+L +3V3-RESCUE-SUPER_UART_front #PWR067
 U 1 1 5943325E
 P 6100 5100
-F 0 "#PWR061" H 6130 5130 10  0001 C CNN
+AR Path="/5943325E" Ref="#PWR067"  Part="1"
+AR Path="/5933A622/5943325E" Ref="#PWR067"  Part="1"
+F 0 "#PWR067" H 6130 5130 10  0001 C CNN
 F 1 "+3V3" H 6100 5230 50  0000 C CNN
 F 2 "" H 6100 5100 50  0001 C CNN
@@
 $EndComp
 $Comp
-L +3V3 #PWR062
+L +3V3-RESCUE-SUPER_UART_front #PWR068
 U 1 1 59433264
 P 5700 5100
-F 0 "#PWR062" H 5730 5130 10  0001 C CNN
+AR Path="/59433264" Ref="#PWR068"  Part="1"
+AR Path="/5933A622/59433264" Ref="#PWR068"  Part="1"
+F 0 "#PWR068" H 5730 5130 10  0001 C CNN
 F 1 "+3V3" H 5700 5230 50  0000 C CNN
 F 2 "" H 5700 5100 50  0001 C CNN
@@
 P 5400 5450
 F 0 "RN3" V 5300 5450 60  0000 C CNN
-F 1 "R" V 5400 5450 40  0000 C CNN
+F 1 "1k" V 5400 5450 40  0000 C CNN
 F 2 "niceRLC:4x0603_N" V 5550 5450 30  0001 C CNN
 F 3 "" H 5400 5450 30  0000 C CNN
@@
 P 5400 5550
 F 0 "RN3" V 5350 5300 40  0001 C CNN
-F 1 "R" V 5400 5550 40  0000 C CNN
+F 1 "1k" V 5400 5550 40  0000 C CNN
 F 2 "niceRLC:4x0603_N" V 5550 5550 30  0001 C CNN
 F 3 "" H 5400 5550 30  0000 C CNN
@@
 P 5400 6600
 F 0 "RN3" V 5350 6350 40  0001 C CNN
-F 1 "R" V 5400 6600 40  0000 C CNN
+F 1 "1k" V 5400 6600 40  0000 C CNN
 F 2 "niceRLC:4x0603_N" V 5550 6600 30  0001 C CNN
 F 3 "" H 5400 6600 30  0000 C CNN
@@
 	4850 6600 5250 6600
 $Comp
-L +3V3 #PWR063
+L +3V3-RESCUE-SUPER_UART_front #PWR069
 U 1 1 59433291
 P 6100 5950
-F 0 "#PWR063" H 6130 5980 10  0001 C CNN
+AR Path="/59433291" Ref="#PWR069"  Part="1"
+AR Path="/5933A622/59433291" Ref="#PWR069"  Part="1"
+F 0 "#PWR069" H 6130 5980 10  0001 C CNN
 F 1 "+3V3" H 6100 6080 50  0000 C CNN
 F 2 "" H 6100 5950 50  0001 C CNN
@@
 $EndComp
 $Comp
-L +3V3 #PWR064
+L +3V3-RESCUE-SUPER_UART_front #PWR070
 U 1 1 59433297
 P 5600 6000
-F 0 "#PWR064" H 5630 6030 10  0001 C CNN
+AR Path="/59433297" Ref="#PWR070"  Part="1"
+AR Path="/5933A622/59433297" Ref="#PWR070"  Part="1"
+F 0 "#PWR070" H 5630 6030 10  0001 C CNN
 F 1 "+3V3" H 5600 6130 50  0000 C CNN
 F 2 "" H 5600 6000 50  0001 C CNN
@@
 P 5350 6350
 F 0 "RN3" V 5300 6100 40  0001 C CNN
-F 1 "R" V 5350 6350 40  0000 C CNN
+F 1 "1k" V 5350 6350 40  0000 C CNN
 F 2 "niceRLC:4x0603_N" V 5500 6350 30  0001 C CNN
 F 3 "" H 5350 6350 30  0000 C CNN
@@
 	4900 3050 4900 3250
 $Comp
-L +3V3 #PWR065
+L +3V3-RESCUE-SUPER_UART_front #PWR071
 U 1 1 594889A8
 P 4900 2700
-F 0 "#PWR065" H 4930 2730 10  0001 C CNN
+AR Path="/594889A8" Ref="#PWR071"  Part="1"
+AR Path="/5933A622/594889A8" Ref="#PWR071"  Part="1"
+F 0 "#PWR071" H 4930 2730 10  0001 C CNN
 F 1 "+3V3" H 4900 2830 50  0000 C CNN
 F 2 "" H 4900 2700 50  0001 C CNN
@@
 	5800 3050 5800 2550
 $Comp
-L GND #PWR066
+L GND #PWR072
 U 1 1 59488CCB
 P 4900 3500
-F 0 "#PWR066" H 4930 3470 10  0001 C CNN
+F 0 "#PWR072" H 4930 3470 10  0001 C CNN
 F 1 "GND" H 4900 3375 40  0001 C CNN
 F 2 "" H 4900 3500 50  0001 C CNN
@@
 Text HLabel 4400 2900 0    56   Input ~ 0
 ~VDD1_EN
+Text Notes 8800 2050 0    56   ~ 0
+Add some ESD caps
 $EndSCHEMATC
