File: kicad/main/SUPER_UART_main.kicad_pcb (KiCad board)
At the start: 2 copper layers, 100 x 35 mm, 91 parts, among them CON1 PIN-1x6, CON2 PIN-1x6, CON3 PIN-1x6, CON4 PIN-1x6, CON5 PIN-2x5, CON6 PIN-2x5, SW1 5V, SW10 TX, SW11 ISO, SW12 I2C, SW13 SPI, SW14 I2C, SW15 SPI, SW16 DTR, SW17 RTS, SW18 SPY, SW2 3V3, SW3 2V5, SW4 1V8, SW5 5V, SW6 3V3, SW7 2V5, SW8 1V8, SW9 RX, U1 SN74LVC2T45DCTT, U2 SN74LVC2T45DCTT, U3 SN74LVC2T45DCTT, U4 SN74LVC2T45DCTT, U5 SN74LVC2T45DCTT, U6 SN74LVC2T45DCTT, U7 SN74LVC2T45DCTT, U8 SN74LVC2T45DCTT

Commit message: Add missing files
Parts:
- removed CON6: PIN-2x5, pnIDC:IDC10_a
- removed D10, D14, D18, D22: RXD, pnSemiconductor:LED0603_R
- removed D11, D15, D19, D23: TXD, pnSemiconductor:LED0603_R
- removed D12, D16, D20, D24: CTS, pnSemiconductor:LED0603_R
- removed D13, D17, D21, D9: DTR, pnSemiconductor:LED0603_R
- removed D25, D26, D27, D28, D3, D4, D5, D6, D7, D8: PESD5V2S2UT, SOT23-3_N
- removed D29: DSR, pnSemiconductor:LED0603_R
- removed D30: RTS, pnSemiconductor:LED0603_R
- removed D31: RI, pnSemiconductor:LED0603_R
- removed D32: DCD, pnSemiconductor:LED0603_R
- removed RN1, RN2, RN3, RN4: R, pnRLC:4x0603_N
- removed RN5, RN6, RN7, RN8, RN9: R, 4x0603_N
- removed SW1, SW5: 5V, pnSwitches:TACTB-64K-F
- removed SW10: TX, pnSwitches:TACTB-64K-F
- removed SW11: ISO, pnSwitches:TACTB-64K-F
- removed SW12, SW14: I2C, pnSwitches:TACTB-64K-F
- removed SW13, SW15: SPI, pnSwitches:TACTB-64K-F
- removed SW16: DTR, pnSwitches:TACTB-64K-F
- removed SW17: RTS, pnSwitches:TACTB-64K-F
- removed SW18: SPY, pnSwitches:TACTB-64K-F
- removed SW2, SW6: 3V3, pnSwitches:TACTB-64K-F
- removed SW3, SW7: 2V5, pnSwitches:TACTB-64K-F
- removed SW4, SW8: 1V8, pnSwitches:TACTB-64K-F
- removed SW9: RX, pnSwitches:TACTB-64K-F
- removed U8: SN74LVC2T45DCTT, niceSemiconductors:TI_SSOP-8_N
- added C18: 100n, 0603_N, F.Cu at (61.2, 28.8)
- added C19: 100n, 0603_N, F.Cu at (60.0, 46.5)
- added C20: 100n, 0603_N, F.Cu at (49.9, 42.0)
- added C21: 10u, niceRLC:0805_N, F.Cu at (79.3, 45.4)
- added C22: 1u, 0603_N, F.Cu at (77.5, 45.4)
- added C23: 1u, 0603_N, F.Cu at (71.5, 45.4)
- added C24: 10u, niceRLC:0805_N, F.Cu at (69.7, 45.4)
- added C25: 100n, 0603_N, F.Cu at (94.5, 42.1)
- added C26: 100n, 0603_N, F.Cu at (43.2, 33.9)
- added C27: 100n, 0603_N, F.Cu at (28.8, 42.0)
- added C28: 100n, 0603_N, F.Cu at (39.7, 43.5)
- added C29: 10u, niceRLC:0805_N, F.Cu at (35.9, 54.6)
- added J1: USB_B, Connectors:USB_B, F.Cu at (86.4, 28.5)
- added MECH2: case, pnMechanical:frog, B.Cu at (67.7, 38.6)
- added Q1: 12MHz, XT3.2x2.5_N, F.Cu at (69.3, 36.0)
- added R1: 24R, 0603_R_N, F.Cu at (86.5, 34.4)
- added R10: 10k, 0603_R_N, F.Cu at (97.5, 43.1)
- added R11: 22k, 0603_R_N, F.Cu at (90.8, 45.6)
- added R12: 10k, 0603_R_N, F.Cu at (60.0, 27.6)
- added R13: 10k, 0603_R_N, F.Cu at (113.4, 29.9)
- added R14: 10k, 0603_R_N, F.Cu at (103.4, 44.9)
- added R15: 10k, 0603_R_N, F.Cu at (74.6, 38.1)
- added R2: 24R, 0603_R_N, F.Cu at (75.5, 34.4)
- added R3: 24R, 0603_R_N, F.Cu at (86.5, 32.8)
- added R4: 24R, 0603_R_N, F.Cu at (75.5, 32.8)
- added R5: 12k, 0603_R_N, F.Cu at (64.8, 32.3)
- added R6: FERR, 0603_R_N, F.Cu at (65.5, 26.1)
- added R7: FERR, 0603_R_N, F.Cu at (69.2, 30.6)
- added R8: 10k, 0603_R_N, F.Cu at (97.5, 46.1)
- added R9: 10k, 0603_R_N, F.Cu at (91.5, 43.4)
- added REL1: V23026, pnRelay:V23026, F.Cu at (102.6, 23.8)
- added T1: N-MOS_small, SOT23-3_N, F.Cu at (113.4, 27.3)
- added T2: N-MOS_small, SOT23-3_N, F.Cu at (103.4, 42.3)
- added TP1: Testpoint, pnConnector:TP_1mm, F.Cu at (117.0, 49.0)
- added TP2: Testpoint, pnConnector:TP_1mm, F.Cu at (71.5, 47.7)
- added TP3: Testpoint, pnConnector:TP_1mm, F.Cu at (76.5, 47.2)
- added TP4: Testpoint, pnConnector:TP_1mm, F.Cu at (77.5, 43.1)
- added TP5: Testpoint, pnConnector:TP_1mm, F.Cu at (30.3, 30.5)
- added X1: BUZZER, pnOther:buzzer_12x9.0, F.Cu at (111.9, 41.8)
- C1, C8, C9: value 100n -> 10u; footprint 0603_N -> niceRLC:0805_N; moved to F.Cu
- C10, C11, C12, C13, C14, C15, C16, C17, C2, C3, C4, C5: moved to F.Cu
- C6, C7: value 100n -> 22p; moved to F.Cu
- CON1: value PIN-1x6 -> PIN-2x4; footprint pnConnector:NIGINI_NCDW-06 -> nicePinheaders:PIN-2x4_F_angled_N
- CON2: value PIN-1x6 -> PIN-2x2; footprint pnConnector:NIGINI_NCDW-06 -> nicePinheaders:PIN-2x2_F_angled_N
- CON3: value PIN-1x6 -> PIN-2x5; footprint pnConnector:NIGINI_NCDW-06 -> nicePinheaders:PIN-2x5_F_angled_N
- CON4: value PIN-1x6 -> PIN-2x12; footprint pnConnector:NIGINI_NCDW-06 -> nicePinheaders:PIN-2x12_F_angled_N
- CON5: value PIN-2x5 -> JTAG; footprint pnConnector:DB9MV -> PIN-1x6_N
- D1, D2: value PESD5V2S2UT -> BAS70; moved to F.Cu
- MECH1: value dummy -> case; footprint niceMechanical:dummy -> dummy
- U1: value SN74LVC2T45DCTT -> ADuM3160; footprint niceSemiconductors:TI_SSOP-8_N -> SOIC-16_N; moved to F.Cu
- U2: value SN74LVC2T45DCTT -> FT4232HL_UART; footprint niceSemiconductors:TI_SSOP-8_N -> niceSemiconductors:FTDI_LQFP64_M; moved to F.Cu
- U3: value SN74LVC2T45DCTT -> USBLC6-2SC6; footprint niceSemiconductors:TI_SSOP-8_N -> SOT23-6_N; moved to F.Cu
- U4: value SN74LVC2T45DCTT -> AM1S-0505SZ; footprint niceSemiconductors:TI_SSOP-8_N -> niceModules:AM1S-Z_N; moved to F.Cu
- U5: value SN74LVC2T45DCTT -> MIC5504-3.3YM5-TR; footprint niceSemiconductors:TI_SSOP-8_N -> niceSemiconductors:SOT23-5_N; moved to F.Cu
- U6: value SN74LVC2T45DCTT -> 93LC46BT-I/OT; footprint niceSemiconductors:TI_SSOP-8_N -> niceSemiconductors:SOT23-6_N; moved to F.Cu
- U7: value SN74LVC2T45DCTT -> XC9536XL-10VQG64; footprint niceSemiconductors:TI_SSOP-8_N -> Xilinx_VQFP64_M; moved to F.Cu
- moved CON5 120.9 mm to (30.6, 24.5), turned to 270 degrees
- moved CON1 109.2 mm to (26.0, 55.9), turned to 90 degrees
- moved C17 101.4 mm to (66.2, 40.5), turned to 315 degrees
- moved U7 90.3 mm to (35.0, 36.9), turned to 225 degrees
- moved U2 89.7 mm to (57.2, 37.1), turned to 225 degrees
- moved C13 85.0 mm to (48.6, 33.4), turned to 135 degrees
- moved C6 83.9 mm to (67.9, 38.8), turned to 315 degrees
- moved C16 80.7 mm to (52.8, 29.2), turned to 135 degrees
- moved C5 80.7 mm to (76.2, 41.1), turned to 90 degrees
- moved C15 80.5 mm to (51.6, 43.8), turned to 225 degrees
- moved C10 79.1 mm to (62.4, 29.9), turned to 45 degrees
- moved C7 77.5 mm to (67.1, 34.6), turned to 225 degrees
- moved C14 77.2 mm to (63.3, 43.3), turned to 315 degrees
- moved C8 76.3 mm to (63.9, 27.2), turned to 135 degrees
- moved CON2 75.0 mm to (40.0, 55.9)
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Connections:
- C1 pad 1: VDD -> ISO_VDD
- C1 pad 2: GND -> ISO_GND
- C10 pad 1: +3V3 -> /VPLL
- C11 pad 1: +3V3 -> /VPHY
- C12 pad 1: VDD -> +3V3
- C13 pad 1: VDD -> +3V3
- C14 pad 1: VDD -> +3V3
- C17 pad 1: ISO_VDD -> +1V8
- C17 pad 2: ISO_GND -> GND
- C2 pad 1: +3V3 -> ISO_VDD
- C2 pad 2: GND -> ISO_GND
- C3 pad 1: +3V3 -> Net-(C3-Pad1)
- C3 pad 2: GND -> ISO_GND
- C4 pad 1: ISO_VDD -> Net-(C4-Pad1)
- C4 pad 2: ISO_GND -> GND
- C5 pad 1: ISO_VDD -> +5V
- C5 pad 2: ISO_GND -> GND
- C6 pad 1: ISO_3V3 -> Net-(C6-Pad1)
- C6 pad 2: ISO_GND -> GND
- C7 pad 1: ISO_3V3 -> Net-(C7-Pad1)
- C7 pad 2: ISO_GND -> GND
- C8 pad 1: VDD -> /VPLL
- C9 pad 1: VDD -> /VPHY
- CON1 pad 1: DTR_A -> GND
- CON1 pad 2: RXD_A -> GND
- CON1 pad 3: TXD_A -> /~CTS_A_OC
- CON1 pad 4: ISO_VDD -> /RXD_A
- CON1 pad 5: CTS_A -> /TXD_C
- CON1 pad 6: ISO_GND -> /CTS_A
- CON2 pad 1: DTR_B -> +5V
- CON2 pad 2: RXD_B -> +5V
- CON2 pad 3: TXD_B -> GND
- CON2 pad 4: VDD -> GND
- CON3 pad 1: DTR_C -> /AUX1
- CON3 pad 2: RXD_C -> (no net)
- CON3 pad 3: TXD_C -> /~RXD_A_OC
- CON3 pad 4: VDD -> (no net)
- CON3 pad 5: CTS_C -> /CTS_C
- CON3 pad 6: GND -> /DTR_B
- CON4 pad 1: DTR_D -> /SR_LOAD
- CON4 pad 2: RXD_D -> /~USB_SUSPEND
- CON4 pad 3: TXD_D -> /~RXD_B_OC
- CON4 pad 4: VDD -> /RXD_B
- CON4 pad 5: CTS_D -> /SR_DATA
- CON4 pad 6: GND -> /SR_CLK
- CON5 pad 1: (no net) -> +3V3
- CON5 pad 2: (no net) -> GND
- CON5 pad 3: (no net) -> /TCK
- CON5 pad 4: (no net) -> /TDO
- CON5 pad 5: (no net) -> /TDI
- CON5 pad 6: (no net) -> /TMS
- D1 pad 1: DTR_A -> Net-(D1-Pad1)
- D1 pad 2: TXD_A -> (no net)
- D1 pad 3: ISO_GND -> +5V
- D2 pad 1: RXD_A -> Net-(D2-Pad1)
- D2 pad 2: CTS_A -> (no net)
- D2 pad 3: ISO_GND -> +5V
- U1 pad 2: Net-(RN1-Pad7) -> ISO_GND
- U1 pad 3: Net-(RN1-Pad8) -> Net-(C3-Pad1)
- U1 pad 4: ISO_GND -> Net-(C3-Pad1)
- U1 pad 5: ISO_GND -> Net-(C3-Pad1)
- U1 pad 6: (no net) -> Net-(R1-Pad2)
- U1 pad 7: (no net) -> Net-(R3-Pad2)
- U1 pad 8: ISO_3V3 -> ISO_GND
- U2 pad 1: ISO_3V3 -> GND
- U2 pad 2: (no net) -> Net-(C6-Pad1)
- U2 pad 3: (no net) -> Net-(C7-Pad1)
- U2 pad 4: ISO_GND -> /VPHY
- U2 pad 5: ISO_GND -> GND
- U2 pad 7: Net-(RN1-Pad6) -> /D-
- U2 pad 8: ISO_VDD -> /D+
- U3 pad 1: VDD -> /ISO_D-
- U3 pad 2: Net-(RN2-Pad7) -> ISO_GND
- U3 pad 3: Net-(RN2-Pad8) -> /ISO_D+
- U3 pad 4: GND -> /ISO_D+
- U3 pad 5: GND -> ISO_VDD
- U3 pad 6: (no net) -> /ISO_D-
- U4 pad 1: +3V3 -> ISO_GND
- U4 pad 2: (no net) -> ISO_VDD
- U4 pad 3: (no net) -> GND
- U4 pad 4: GND -> +5V
- U5 pad 1: VDD -> +5V
- U5 pad 2: Net-(RN3-Pad7) -> GND
- U5 pad 3: Net-(RN3-Pad8) -> +5V
- U5 pad 4: GND -> (no net)
- U5 pad 5: GND -> +3V3
- U6 pad 1: +3V3 -> Net-(R11-Pad2)
- U6 pad 2: (no net) -> GND
- U6 pad 3: (no net) -> /EEDATA
- U6 pad 4: GND -> /EECLK
- U6 pad 5: GND -> /EECS
- U6 pad 6: Net-(RN3-Pad5) -> +3V3
- U7 pad 1: VDD -> (no net)
- U7 pad 2: Net-(RN4-Pad7) -> /FTDI_RXD_C
- U7 pad 3: Net-(RN4-Pad8) -> +3V3
- U7 pad 4: GND -> (no net)
- U7 pad 5: GND -> /FTDI_DTR_B
- U7 pad 6: (no net) -> /FTDI_CTS_B
- U7 pad 7: (no net) -> /FTDI_RTS_B
- U7 pad 8: +3V3 -> /FTDI_RXD_B
Routing:
- net GND: track 41.0 -> 385.8 mm, vias 12 -> 97
- net +5V: track 0.00 -> 198.3 mm, vias 0 -> 7
- net +3V3: track 16.3 -> 188.0 mm, vias 6 -> 10
- net /AUX1: track 0.00 -> 129.1 mm, vias 0 -> 3
- net /OPTO_EN: track 0.00 -> 124.5 mm, vias 0 -> 2
- net /FTDI_RESET: track 0.00 -> 111.0 mm, vias 0 -> 4
- net /BUZZER: track 0.00 -> 96.2 mm, vias 0 -> 2
- net /~USB_SUSPEND: track 0.00 -> 91.1 mm, vias 0 -> 2
- net /TXD_D: track 0.00 -> 80.5 mm
- net /RXD_D: track 0.00 -> 79.7 mm
- net /EECS: track 0.00 -> 77.5 mm
- net /SR_CLK: track 0.00 -> 75.5 mm
- net /EECLK: track 0.00 -> 72.5 mm, vias 0 -> 2
- net /CTS_B: track 0.00 -> 68.1 mm
- net /TXD_B: track 0.00 -> 68.0 mm
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- added copper zone on F.Cu, net +1V8
- added copper zone on F.Cu, net +3V3
- added copper zone on F.Cu, net +5V
- added copper zone on B.Cu, net GND
- added copper zone on F.Cu, net GND
- added copper zone on B.Cu, net ISO_GND
- added copper zone on F.Cu, net ISO_GND
- added copper zone on F.Cu, net ISO_VDD
Other:
- board size 100 x 35 mm -> 100 x 43 mm
- net class Default: clearance 0.1524 -> 0.17
- net class IO added: clearance 0.25, trace_width 0.1524, via_dia 0.6048, via_drill 0.3
- net class USB added: clearance 0.1524, trace_width 0.5, via_dia 0.6048, via_drill 0.3
- rule trace_clearance: 0.1524 -> 0.17
- board text added: "2"
- board text added: "3"
- board text added: "NOP041"
- board text added: "http://nicecircuits.com/uart/"
- board text added: "niceUART"
